File: BatteryMonitor.kicad_sch (KiCad schematic)
At the start: 1 part

Commit message: feat: resolved splitting cells across monitor
Connections:
- net VIN_MONITOR: now reaches U?.1 (V+)
- net C12: now reaches U?.2 (C12), U?.4 (C11), U?.6 (C10)
- net C1_IN renamed C1
- net C2_IN renamed C2
- net C3_IN renamed C3
- net C6_IN renamed C6
- net C7_IN renamed C7
- net C8_IN renamed C8
- net C9_IN renamed C9
Other:
- moved on the sheet: U?
