File: bms-kicad-project/FilteringCells.kicad_sch (KiCad schematic)
At the start: 48 parts, among them J1 S7B-XH-A, Q1 BSS308PE_H6327, Q2 BSS308PE_H6327, Q3 BSS308PE_H6327, Q5 BSS308PE_H6327, Q6 BSS308PE_H6327, Q7 BSS308PE_H6327

Commit message: feat: add breakout board templates for filtering circuit resistors
Other:
- company: AeroNU FixedWing -> AeroNU - FixedWing
Changed lines of the file:
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@@
     (date "2024-03-29")
     (rev "1")
-    (company "AeroNU FixedWing")
+    (company "AeroNU - FixedWing")
   )
   (junction (at 80.01 179.07) (diameter 0) (color 0 0 0 0)
