File: bms-kicad-project/bms-board.kicad_pcb (KiCad board)
At the start: 4 copper layers, 240 parts, among them J1 12402012E212A, J2 DEBUG, J3 Conn_02x18_Odd_Even, J4 Conn_02x18_Odd_Even, K1 G6L-1P_DC5, Q1 BSS308PE_H6327, Q10 BSS308PE_H6327, Q11 BSS308PE_H6327, Q12 BSS308PE_H6327, Q13 BSS308PE_H6327, Q14 BSS308PE_H6327, Q2 BSS308PE_H6327, Q3 BSS308PE_H6327, Q4 BSS308PE_H6327, Q5 BSS308PE_H6327, Q6 BSS308PE_H6327, Q7 BSS308PE_H6327, Q8 BSS308PE_H6327, Q9 BSS308PE_H6327, SW1 KMR223G LFG, SW2 KMR223G LFG, U1 LTC6804-2, U2 W25Q128JVSIQ TR, U3 NCP1117ST33T3G, U4 RP2040, U5 SIC461ED-T1-GE3, U6 TPS61170DRVR, U7 SN74LVC1G17DCKR, X1 ABM8-272-T3

Commit message: feat: Just shifting a few things around
Parts:
- added C64: 0.1µ, FixedWing:G-21_MUR, F.Cu at (113.0, 88.9)
- added C65: 1.5n, FixedWing:G-21_MUR, F.Cu at (113.0, 91.8)
- added C66: 0.1µ, FixedWing:G-21_MUR, F.Cu at (113.0, 94.7)
- added J10: XT60PW-F, FixedWing:XT60PWF, F.Cu at (74.5, 72.6)
- added J11: 1053131302, FixedWing:105313YY02, F.Cu at (114.8, 37.8)
- added J12: XT60PW-F, FixedWing:XT60PWF, F.Cu at (74.5, 93.1)
- added J13: 1053131302, FixedWing:105313YY02, F.Cu at (124.9, 37.8)
- added J14: 1053131303, FixedWing:105313YY03, F.Cu at (97.1, 90.1)
- added J15: XT60PW-F, FixedWing:XT60PWF, F.Cu at (74.5, 113.6)
- added J16: SM06B-GHS-TB, FixedWing:SM06B-GHS-TB, F.Cu at (89.4, 108.4)
- added J17: 5024940670, FixedWing:5024940670, F.Cu at (117.7, 72.7)
- added J5: Conn_02x18_Odd_Even, Connector_PinHeader_2.54mm:PinHeader_2x18_P2.54mm_Vertical, F.Cu at (140.4, 37.6)
- added J6: XT60PW-F, FixedWing:XT60PWF, F.Cu at (74.5, 52.1)
- added J7: 1053131302, FixedWing:105313YY02, F.Cu at (94.6, 37.8)
- added J8: XT60PW-M, FixedWing:XT60PWM, F.Cu at (98.3, 83.9)
- added J9: 1053131302, FixedWing:105313YY02, F.Cu at (104.7, 37.8)
- added LED14: LTST-C170KGKT, FixedWing:LED_LTST-C170KGKT_LTO, F.Cu at (98.7, 139.4)
- added LED15: COM-16347, FixedWing:COM-16347_SPK, F.Cu at (119.0, 90.8)
- added R107: 56.2k, FixedWing:RC0805N_YAG, F.Cu at (89.9, 132.0)
- added R108: 5.6k, FixedWing:RESC2012X60N, F.Cu at (103.4, 98.5)
- added R109: 100, FixedWing:RESC2012X50N, F.Cu at (125.2, 89.0)
- added R110: 100, FixedWing:RESC2012X50N, F.Cu at (125.2, 92.1)
- added R111: 100k, FixedWing:RESC2012X60N, F.Cu at (103.4, 101.5)
- added U8: ACS72981KLRATR-150B5, FixedWing:ACS780LLRTR050BT, F.Cu at (106.0, 92.3)
- C14: value 0.1µ -> 4.7u; footprint FixedWing:CAP_GCJ-18_MUR -> FixedWing:CAPC2012X145N
- C15: value 15p -> 4.7u; footprint FixedWing:CAPC2012X70 -> FixedWing:CAPC2012X145N
- C16: value 15p -> 33n; footprint FixedWing:CAPC2012X70 -> FixedWing:CAPC2012X94N
- C17: value 0.1µ -> 33n; footprint FixedWing:CAP_GCJ-18_MUR -> FixedWing:CAPC2012X94N
- C18, C19, C20: value 10µ -> 4.7u; footprint FixedWing:CAP_CL21B106KOQNNNE_SAM -> FixedWing:CAPC2012X145N
- C22: value 0.1µ -> 15p; footprint FixedWing:CAP_GCJ-18_MUR -> FixedWing:CAPC2012X70
- C23: value 1µ -> 15p; footprint FixedWing:CAPC2012X140N -> FixedWing:CAPC2012X70
- C25: value 1µ -> 10µ; footprint FixedWing:CAPC2012X140N -> FixedWing:CAP_CL21B106KOQNNNE_SAM
- C26, C27: value 0.1µ -> 10µ; footprint FixedWing:CAP_GCJ-18_MUR -> FixedWing:CAP_CL21B106KOQNNNE_SAM
- C30: value 0.1µ -> 1µ; footprint FixedWing:CAP_GCJ-18_MUR -> FixedWing:CAPC2012X140N
- C32: value 220u -> 1µ; footprint FixedWing:CAPPRD500W60D1000H2500 -> FixedWing:CAPC2012X140N
- C34: value 560p -> 0.1µ; footprint FixedWing:CAP_CC0805_YAG -> FixedWing:CAP_GCJ-18_MUR
- C35: value 1u -> 0.1µ; footprint FixedWing:CAPC1608X90N -> FixedWing:CAP_GCJ-18_MUR
- C36: value 33n -> 0.1µ; footprint FixedWing:CAPC2012X94N -> FixedWing:CAP_GCJ-18_MUR
- C37: value 4.7u -> 0.1µ; footprint FixedWing:CAPC2012X145N -> FixedWing:CAP_GCJ-18_MUR
- C38: value 3.9n -> 0.1µ; footprint FixedWing:G-21_MUR -> FixedWing:CAP_GCJ-18_MUR
- C39: value 0.1µ -> 220u; footprint FixedWing:CAP_GCJ-18_MUR -> FixedWing:CAPPRD500W60D1000H2500
- C40: value 1.5n -> 0.1µ; footprint FixedWing:G-21_MUR -> FixedWing:CAP_GCJ-18_MUR
- C41: value C -> 560p; footprint Capacitor_SMD:C_0805_2012Metric -> FixedWing:CAP_CC0805_YAG
- C42: value 0.1µ -> 1u; footprint FixedWing:CAP_GCJ-18_MUR -> FixedWing:CAPC1608X90N
- C43: value 47u -> 33n; footprint FixedWing:G-32_MUR -> FixedWing:CAPC2012X94N
- C44: value 47u -> 4.7u; footprint FixedWing:G-32_MUR -> FixedWing:CAPC2012X145N
- C45: value 47u -> 3.9n; footprint FixedWing:G-32_MUR -> FixedWing:G-21_MUR
- C46, C49: value 47u -> 0.1µ; footprint FixedWing:G-32_MUR -> FixedWing:CAP_GCJ-18_MUR
- C47: value 47u -> 1.5n; footprint FixedWing:G-32_MUR -> FixedWing:G-21_MUR
- C48: value 47u -> C; footprint FixedWing:G-32_MUR -> Capacitor_SMD:C_0805_2012Metric
- C57, C58, C59, C60, C61: value 4.7u -> 47u; footprint FixedWing:CAPC2012X145N -> FixedWing:G-32_MUR
- C62, C63: value 33n -> 47u; footprint FixedWing:CAPC2012X94N -> FixedWing:G-32_MUR
- D2, D3: value CMHD4448 -> 1N4448X-TP; footprint FixedWing:CR_SOD-123F_CNS -> FixedWing:1N4448XTP
- J1: value 12402012E212A -> S13B-XH-A; footprint FixedWing:AMPHENOL_12402012E212A -> FixedWing:S13BXHALFSN
- J2: value DEBUG -> 12402012E212A; footprint Connector_PinHeader_2.54mm:PinHeader_1x03_P2.54mm_Vertical -> FixedWing:AMPHENOL_12402012E212A
- J3: value Conn_02x18_Odd_Even -> DEBUG; footprint Connector_PinHeader_2.54mm:PinHeader_2x18_P2.54mm_Vertical -> Connector_PinHeader_2.54mm:PinHeader_1x03_P2.54mm_Vertical
- L15: value 600Ω -> SDR0302-120ML; footprint FixedWing:IND_BLM31PG391SN1L_MUR -> FixedWing:SDR0302-471KL
- L16: value 5.6u -> 600Ω; footprint FixedWing:IND_IHLP-6767GZ_VIS -> FixedWing:IND_BLM31PG391SN1L_MUR
- L17: value SDR0302-120ML -> 5.6u; footprint FixedWing:SDR0302-471KL -> FixedWing:IND_IHLP-6767GZ_VIS
- R100: value 11k5 -> 1k
- R101: value 100k -> 93.1k
- R102: value 56k2 -> 3.3; footprint FixedWing:RC0805N_YAG -> FixedWing:RESC1608X55N
- R103: value 33k2 -> 10k; footprint FixedWing:RC0805N_YAG -> FixedWing:KOA_Speer-RK73H2A-0-0-MFG
- R104: value 33k2 -> 11.5k
- R105: value 56k2 -> R; footprint FixedWing:RC0805N_YAG -> Resistor_SMD:R_0805_2012Metric
- R106: value 10k -> R; footprint FixedWing:KOA_Speer-RK73H2A-0-0-MFG -> Resistor_SMD:R_0805_2012Metric
- R75: value 5.6k -> 56k2; footprint FixedWing:RESC2012X60N -> FixedWing:RC0805N_YAG
- R76: value 100 -> 33k2; footprint FixedWing:RESC2012X50N -> FixedWing:RC0805N_YAG
- R77: value 5.6k -> 10k; footprint FixedWing:RESC2012X60N -> FixedWing:KOA_Speer-RK73H2A-0-0-MFG
- R78: value 5.6k -> 33k2; footprint FixedWing:RESC2012X60N -> FixedWing:RC0805N_YAG
- R79: value 1k -> 11k5
- R80: value 1k -> 56k2
- R81: value 5.6k -> 100k
- R82: value 27 -> 5.6k; footprint FixedWing:RC0805N_YAG -> FixedWing:RESC2012X60N
- R83: value 27 -> 100; footprint FixedWing:RC0805N_YAG -> FixedWing:RESC2012X50N
- R84: value 562k -> 5.6k
- R85: value 100k -> 5.6k
- R86: value 100k -> 1k; footprint FixedWing:RESC2012X60N -> FixedWing:RC0805N_YAG
- R87: value 523k -> 1k
- R88: value 10k -> 5.6k; footprint FixedWing:KOA_Speer-RK73H2A-0-0-MFG -> FixedWing:RESC2012X60N
- R89: value 1k -> 27
- R90: value 41.2 -> 27; footprint FixedWing:RC0805N_VIS -> FixedWing:RC0805N_YAG
- R91: value 0 -> 475; footprint FixedWing:RC1206N_YAG -> FixedWing:RESC2012X50N
- R92: value 1k -> 562k; footprint FixedWing:RC0805N_YAG -> FixedWing:RESC2012X60N
- R93: value 93.1k -> 100k
- R94: value 3.3 -> 100k; footprint FixedWing:RESC1608X55N -> FixedWing:RESC2012X60N
- R95: value 10k -> 523k; footprint FixedWing:KOA_Speer-RK73H2A-0-0-MFG -> FixedWing:RC0805N_YAG
- R96: value 11.5k -> 10k; footprint FixedWing:RC0805N_YAG -> FixedWing:KOA_Speer-RK73H2A-0-0-MFG
- R97: value R -> 1k; footprint Resistor_SMD:R_0805_2012Metric -> FixedWing:RC0805N_YAG
- R98: value R -> 41.2; footprint Resistor_SMD:R_0805_2012Metric -> FixedWing:RC0805N_VIS
- R99: value 56.2k -> 0; footprint FixedWing:RC0805N_YAG -> FixedWing:RC1206N_YAG
- U1: value LTC6804-2 -> TPS61170DRVR; footprint FixedWing:SSOP-48_5.3x12.8mm_P0.5mm -> FixedWing:DRV6_1P6X1
- U2: value W25Q128JVSIQ TR -> SN74LVC1G17DCKR; footprint FixedWing:SOIC_208MIL_WIN -> FixedWing:DCK5
- U3: value NCP1117ST33T3G -> LTC6804-2; footprint FixedWing:SOT223-3_ONS -> FixedWing:SSOP-48_5.3x12.8mm_P0.5mm
- U4: value RP2040 -> W25Q128JVSIQ TR; footprint FixedWing:RP2040-QFN-56 -> FixedWing:SOIC_208MIL_WIN
- U5: value SIC461ED-T1-GE3 -> NCP1117ST33T3G; footprint FixedWing:CONV_SIC461ED-T1-GE3 -> FixedWing:SOT223-3_ONS
- U6: value TPS61170DRVR -> RP2040; footprint FixedWing:DRV6_1P6X1 -> FixedWing:RP2040-QFN-56
- U7: value SN74LVC1G17DCKR -> SIC461ED-T1-GE3; footprint FixedWing:DCK5 -> FixedWing:CONV_SIC461ED-T1-GE3
- moved C59 109.0 mm to (75.9, 156.6)
- moved R106 108.9 mm to (98.7, 153.9)
- moved C58 108.1 mm to (75.9, 152.5)
- moved C57 107.1 mm to (75.9, 148.3)
- moved C37 102.6 mm to (151.6, 41.6)
- moved C63 101.1 mm to (81.4, 152.5)
- moved C62 100.3 mm to (81.4, 148.3)
- moved C21 99.4 mm to (133.0, 149.2)
- moved C17 95.4 mm to (152.4, 133.4)
- moved R102 95.0 mm to (98.5, 148.0)
- moved U5 94.9 mm to (159.3, 55.4)
- moved R101 93.1 mm to (94.2, 129.4)
- moved C33 92.2 mm to (147.4, 46.7)
- moved C61 90.9 mm to (81.4, 144.2)
- moved C35 90.6 mm to (151.6, 36.5)
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Connections:
- C14 pad 1: Net-(U1-V+) -> GND
- C14 pad 2: GND -> Net-(U1-CTRL)
- C15 pad 2: /RP2040 Microcontroller/XIN -> Net-(U1-CTRL)
- C16 pad 1: GND -> Net-(C16-Pad1)
- C17 pad 1: +3V3 -> GND
- C17 pad 2: GND -> Net-(C16-Pad1)
- C18 pad 1: Net-(D4-K) -> GND
- C18 pad 2: GND -> Net-(D1-K)
- C19 pad 2: +3V3 -> Net-(D1-K)
- C20 pad 2: +3V3 -> Net-(D1-K)
- C21 pad 1: GND -> Net-(U3-V+)
- C21 pad 2: +1V1 -> GND
- C22 pad 2: +1V1 -> /RP2040 Microcontroller/XIN
- C23 pad 2: +1V1 -> Net-(C23-Pad2)
- C25 pad 1: GND -> Net-(D4-K)
- C25 pad 2: +3V3 -> GND
- C26 pad 1: +3V3 -> GND
- C26 pad 2: GND -> +3V3
- C28 pad 1: +3V3 -> GND
- C28 pad 2: GND -> +1V1
- C29 pad 1: +3V3 -> GND
- C29 pad 2: GND -> +1V1
- C30 pad 1: +3V3 -> GND
- C30 pad 2: GND -> +1V1
- C32 pad 1: +BATT -> GND
- C32 pad 2: GND -> +3V3
- C33 pad 1: GND -> +3V3
- C33 pad 2: +BATT -> GND
- C34 pad 2: Net-(C34-Pad2) -> +3V3
- C35 pad 1: Net-(U5-VDD) -> +3V3
- C36 pad 1: GND -> +3V3
- C36 pad 2: Net-(U5-SS) -> GND
- C37 pad 1: GND -> +3V3
- C37 pad 2: Net-(U5-VDRV) -> GND
- C38 pad 1: Net-(U5-VSNS) -> +3V3
- C38 pad 2: Net-(C38-Pad2) -> GND
- C39 pad 1: Net-(C39-Pad1) -> +BATT
- C39 pad 2: Net-(U5-PHASE) -> GND
- C40 pad 1: Net-(C38-Pad2) -> GND
- C40 pad 2: +5V -> +BATT
- C41 pad 1: Net-(C41-Pad1) -> GND
- C41 pad 2: GND -> Net-(C41-Pad2)
- C42 pad 1: GND -> Net-(U7-VDD)
- C42 pad 2: +5V -> GND
- C43 pad 2: +5V -> Net-(U7-SS)
- C44 pad 2: +5V -> Net-(U7-VDRV)
- C45 pad 1: GND -> Net-(U7-VSNS)
- C45 pad 2: +5V -> Net-(C45-Pad2)
- C46 pad 1: GND -> Net-(C46-Pad1)
- C46 pad 2: +5V -> Net-(U7-PHASE)
- C47 pad 1: GND -> Net-(C45-Pad2)
- C48 pad 1: GND -> Net-(C48-Pad1)
- C48 pad 2: +5V -> GND
- C57 pad 2: Net-(D1-K) -> +5V
- C58 pad 2: Net-(D1-K) -> +5V
- C59 pad 2: Net-(U6-CTRL) -> +5V
- C60 pad 2: Net-(U6-CTRL) -> +5V
- C61 pad 2: Net-(D1-K) -> +5V
- C62 pad 1: Net-(C62-Pad1) -> GND
- C62 pad 2: Net-(C62-Pad2) -> +5V
- C63 pad 2: Net-(C62-Pad1) -> +5V
- D2 pad 1: Net-(D2-Pad1) -> Net-(D2-K)
- D2 pad 2: Net-(D1-K) -> +BATT
- D3 pad 1: Net-(D2-Pad1) -> Net-(D2-K)
- D3 pad 2: +BATT -> Net-(D1-K)
- J3 pad 1: GND -> /RP2040 Microcontroller/SWCLK
- J3 pad 2: +3V3 -> GND
- J3 pad 3: GND -> /RP2040 Microcontroller/SWD
- J4 pad 1: /RP2040 Microcontroller/GPIO29_ADC3 -> GND
- J4 pad 10: GND -> /RP2040 Microcontroller/GPIO3
- J4 pad 11: /RP2040 Microcontroller/GPIO24 -> GND
- J4 pad 12: GND -> /RP2040 Microcontroller/GPIO4
- J4 pad 13: /RP2040 Microcontroller/GPIO23 -> GND
- J4 pad 14: GND -> /RP2040 Microcontroller/GPIO5
- J4 pad 15: /RP2040 Microcontroller/GPIO22 -> GND
- J4 pad 16: GND -> /RP2040 Microcontroller/GPIO6
- J4 pad 17: /RP2040 Microcontroller/GPIO21 -> GND
- J4 pad 18: GND -> /RP2040 Microcontroller/GPIO7
- J4 pad 19: /RP2040 Microcontroller/GPIO20 -> GND
- J4 pad 2: GND -> +3V3
- J4 pad 20: GND -> /RP2040 Microcontroller/GPIO8
- J4 pad 21: /RP2040 Microcontroller/GPIO19 -> GND
- J4 pad 22: GND -> /RP2040 Microcontroller/GPIO9
- J4 pad 23: /RP2040 Microcontroller/GPIO18 -> GND
- J4 pad 24: GND -> /RP2040 Microcontroller/GPIO10
- J4 pad 25: /RP2040 Microcontroller/GPIO17 -> GND
- J4 pad 26: GND -> /RP2040 Microcontroller/GPIO11
- J4 pad 27: /RP2040 Microcontroller/GPIO16 -> GND
- J4 pad 28: GND -> /RP2040 Microcontroller/GPIO12
- J4 pad 29: /RP2040 Microcontroller/RUN -> GND
- J4 pad 3: /RP2040 Microcontroller/GPIO28_ADC2 -> GND
- J4 pad 30: GND -> /RP2040 Microcontroller/GPIO13
- J4 pad 31: /RP2040 Microcontroller/SWD -> GND
- J4 pad 32: GND -> /RP2040 Microcontroller/GPIO14
- J4 pad 33: /RP2040 Microcontroller/SWCLK -> GND
- J4 pad 34: GND -> /RP2040 Microcontroller/GPIO15
- J4 pad 4: GND -> /RP2040 Microcontroller/GPIO0
- J4 pad 5: /RP2040 Microcontroller/GPIO27_ADC1 -> GND
- J4 pad 6: GND -> /RP2040 Microcontroller/GPIO1
- J4 pad 7: /RP2040 Microcontroller/GPIO26_ADC0 -> GND
- J4 pad 8: GND -> /RP2040 Microcontroller/GPIO2
- J4 pad 9: /RP2040 Microcontroller/GPIO25 -> GND
- K1 pad 4: Net-(U6-CTRL) -> Net-(U1-CTRL)
- K1 pad 8: /RP2040 Microcontroller/GPIO4 -> /RP2040 Microcontroller/GPIO6
- L1 pad 2: unconnected-(L1-Pad2) -> Net-(J1-Pad13)
- L10 pad 1: unconnected-(L10-Pad1) -> Net-(J1-Pad5)
- L11 pad 2: unconnected-(L11-Pad2) -> Net-(J1-Pad8)
- L12 pad 1: unconnected-(L12-Pad1) -> Net-(J1-Pad6)
- L13 pad 2: unconnected-(L13-Pad2) -> Net-(J1-Pad7)
- L14 pad 2: Net-(L14-Pad2) -> Net-(J1-Pad1)
- L15 pad 1: Net-(L15-Pad1) -> Net-(U1-CTRL)
- L15 pad 2: Net-(D2-Pad1) -> Net-(D1-A)
- L16 pad 1: Net-(U5-SW) -> Net-(L16-Pad1)
- L16 pad 2: +5V -> Net-(D2-K)
- L17 pad 1: Net-(U6-CTRL) -> Net-(U7-SW)
- L17 pad 2: Net-(D1-A) -> +5V
- L2 pad 1: Net-(L14-Pad2) -> Net-(J1-Pad1)
- L3 pad 2: unconnected-(L3-Pad2) -> Net-(J1-Pad12)
- L4 pad 1: unconnected-(L4-Pad1) -> Net-(J1-Pad2)
- L5 pad 2: unconnected-(L5-Pad2) -> Net-(J1-Pad11)
- L6 pad 1: unconnected-(L6-Pad1) -> Net-(J1-Pad3)
- L7 pad 2: unconnected-(L7-Pad2) -> Net-(J1-Pad10)
- L8 pad 1: unconnected-(L8-Pad1) -> Net-(J1-Pad4)
- L9 pad 2: unconnected-(L9-Pad2) -> Net-(J1-Pad9)
- Q13 pad 1: Net-(D4-A) -> Net-(Q13-G)
- Q13 pad 2: Net-(D4-K) -> +5V
- Q13 pad 3: +5V -> Net-(Q13-D)
- Q14 pad 1: Net-(Q14-G) -> Net-(D4-A)
- Q14 pad 2: +5V -> Net-(D4-K)
- Q14 pad 3: Net-(Q14-D) -> +5V
- R100 pad 1: Net-(U6-FB) -> Net-(R100-Pad1)
- R100 pad 2: Net-(D1-K) -> Net-(U7-MODE)
- R101 pad 2: Net-(R101-Pad2) -> Net-(U7-FSW)
- R102 pad 1: Net-(R101-Pad2) -> Net-(U7-BOOT)
- R102 pad 2: Net-(U6-FB) -> Net-(C46-Pad1)
- R103 pad 1: Net-(U6-COMP) -> GND
- R103 pad 2: Net-(C62-Pad2) -> Net-(U7-VFB)
- R104 pad 1: GND -> Net-(U7-SW)
- R104 pad 2: Net-(Q14-G) -> Net-(C45-Pad2)
- R105 pad 1: Net-(Q14-G) -> Net-(U7-SW)
- R105 pad 2: +BATT -> Net-(C48-Pad1)
- R106 pad 1: GND -> Net-(U7-SW)
- R106 pad 2: Net-(Q14-D) -> Net-(C48-Pad1)
- R75 pad 1: /RP2040 Microcontroller/GPIO0 -> Net-(Q13-G)
- R75 pad 2: +5V -> +BATT
- R76 pad 1: Net-(U1-V+) -> GND
- R76 pad 2: Net-(L15-Pad1) -> Net-(Q13-G)
- R77 pad 2: Net-(J1-CC1_B) -> Net-(Q13-D)
- R78 pad 1: GND -> Net-(U1-COMP)
- R78 pad 2: Net-(J1-CC1_A) -> Net-(C16-Pad2)
- R79 pad 1: Net-(C16-Pad2) -> Net-(U1-FB)
- R79 pad 2: /RP2040 Microcontroller/XOUT -> Net-(D1-K)
- R80 pad 1: /RP2040 Microcontroller/~{USB_BOOT} -> Net-(R80-Pad1)
- R80 pad 2: /RP2040 Microcontroller/QSPI_SS -> Net-(U1-FB)
- R81 pad 1: +3V3 -> GND
- R81 pad 2: /RP2040 Microcontroller/~{RESET} -> Net-(R80-Pad1)
- R82 pad 1: Net-(U4-USB_DP) -> /RP2040 Microcontroller/GPIO0
- R82 pad 2: /RP2040 Microcontroller/USB_D+ -> +5V
- R83 pad 1: Net-(U4-USB_DM) -> Net-(U3-V+)
- R83 pad 2: /RP2040 Microcontroller/USB_D- -> Net-(L16-Pad1)
- R84 pad 1: Net-(U5-EN) -> GND
- R84 pad 2: +BATT -> Net-(J2-CC1_B)
- R85 pad 1: Net-(R85-Pad1) -> GND
- R85 pad 2: Net-(U5-EN) -> Net-(J2-CC1_A)
- R86 pad 1: GND -> Net-(C23-Pad2)
- R86 pad 2: Net-(R85-Pad1) -> /RP2040 Microcontroller/XOUT
- R87 pad 1: Net-(C34-Pad2) -> /RP2040 Microcontroller/~{USB_BOOT}
- R87 pad 2: Net-(U5-COMP) -> /RP2040 Microcontroller/QSPI_SS
- R88 pad 1: Net-(U5-VDD) -> +3V3
- R88 pad 2: Net-(LED13-A) -> /RP2040 Microcontroller/~{RESET}
- R89 pad 1: GND -> Net-(U6-USB_DP)
- R89 pad 2: Net-(R89-Pad2) -> /RP2040 Microcontroller/USB_D+
- R90 pad 1: GND -> Net-(U6-USB_DM)
- R90 pad 2: Net-(U5-ILIMIT) -> /RP2040 Microcontroller/USB_D-
- R91 pad 1: Net-(U5-VDD) -> /RP2040 Microcontroller/GPIO25
- R91 pad 2: Net-(U5-ULTRASONIC) -> Net-(LED13-A)
- R92 pad 1: Net-(R89-Pad2) -> Net-(U7-EN)
- R92 pad 2: Net-(U5-MODE) -> +BATT
- R93 pad 1: GND -> Net-(R93-Pad1)
- R93 pad 2: Net-(U5-FSW) -> Net-(U7-EN)
- R94 pad 1: Net-(U5-BOOT) -> GND
- R94 pad 2: Net-(C39-Pad1) -> Net-(R93-Pad1)
- R95 pad 1: GND -> Net-(C41-Pad2)
- R95 pad 2: Net-(U5-VFB) -> Net-(U7-COMP)
- R96 pad 1: Net-(U5-SW) -> Net-(U7-VDD)
- R96 pad 2: Net-(C38-Pad2) -> Net-(LED14-A)
- R97 pad 1: Net-(U5-SW) -> GND
- R97 pad 2: Net-(C41-Pad1) -> Net-(R100-Pad1)
- R98 pad 1: Net-(U5-SW) -> GND
- R98 pad 2: Net-(C41-Pad1) -> Net-(U7-ILIMIT)
- R99 pad 1: Net-(U5-VFB) -> Net-(U7-VDD)
- R99 pad 2: +5V -> Net-(U7-ULTRASONIC)
- U1 pad 1: Net-(U1-V+) -> Net-(U1-FB)
- U1 pad 2: /Battery Stack Monitor/C12 -> Net-(U1-COMP)
- U1 pad 3: /Battery Stack Monitor/S12 -> GND
- U1 pad 4: /Battery Stack Monitor/C11 -> Net-(D1-A)
- U1 pad 5: /Battery Stack Monitor/S11 -> Net-(U1-CTRL)
- U1 pad 6: /Battery Stack Monitor/C10 -> Net-(U1-CTRL)
- U1 pad 7: /Battery Stack Monitor/S10 -> GND
- U2 pad 1: /RP2040 Microcontroller/QSPI_SS -> unconnected-(U2-NC-Pad1)
- U2 pad 2: /RP2040 Microcontroller/QSPI_SD1 -> Net-(Q13-D)
- U2 pad 3: /RP2040 Microcontroller/QSPI_SD2 -> GND
- U2 pad 4: unconnected-(U2-GND-Pad4) -> /RP2040 Microcontroller/GPIO6
- U2 pad 5: /RP2040 Microcontroller/QSPI_SD0 -> +5V
- U3 pad 1: GND -> Net-(U3-V+)
- U3 pad 2: +3V3 -> /Battery Stack Monitor/C12
- U3 pad 3: Net-(D4-K) -> /Battery Stack Monitor/S12
- U4 pad 1: +3V3 -> /RP2040 Microcontroller/QSPI_SS
- U4 pad 2: /RP2040 Microcontroller/GPIO0 -> /RP2040 Microcontroller/QSPI_SD1
- U4 pad 3: /RP2040 Microcontroller/GPIO1 -> /RP2040 Microcontroller/QSPI_SD2
- U4 pad 4: /RP2040 Microcontroller/GPIO2 -> unconnected-(U4-GND-Pad4)
- U4 pad 5: /RP2040 Microcontroller/GPIO3 -> /RP2040 Microcontroller/QSPI_SD0
- U4 pad 6: /RP2040 Microcontroller/GPIO4 -> /RP2040 Microcontroller/QSPI_SCLK
- U4 pad 7: /RP2040 Microcontroller/GPIO5 -> /RP2040 Microcontroller/QSPI_SD3
- U4 pad 8: /RP2040 Microcontroller/GPIO6 -> +3V3
- U5 pad 1: +BATT -> GND
- U5 pad 2: Net-(LED13-A) -> +3V3
- U5 pad 3: Net-(U5-EN) -> Net-(D4-K)
- U6 pad 1: Net-(U6-FB) -> +3V3
- U6 pad 2: Net-(U6-COMP) -> /RP2040 Microcontroller/GPIO0
- U6 pad 3: GND -> /RP2040 Microcontroller/GPIO1
- U6 pad 4: Net-(D1-A) -> /RP2040 Microcontroller/GPIO2
- U6 pad 5: Net-(U6-CTRL) -> /RP2040 Microcontroller/GPIO3
- U6 pad 6: Net-(U6-CTRL) -> /RP2040 Microcontroller/GPIO4
- U6 pad 7: GND -> /RP2040 Microcontroller/GPIO5
- U7 pad 1: unconnected-(U7-NC-Pad1) -> +BATT
- U7 pad 2: Net-(Q14-D) -> Net-(LED14-A)
- U7 pad 3: GND -> Net-(U7-EN)
- U7 pad 4: /RP2040 Microcontroller/GPIO4 -> Net-(U7-BOOT)
- U7 pad 5: +5V -> Net-(U7-PHASE)
- X1 pad 3: Net-(C16-Pad2) -> Net-(C23-Pad2)
