File: bms-kicad-project/bms-board.kicad_pcb (KiCad board)
At the start: 4 copper layers, 271 parts, among them J1 S13B-XH-A, J10 XT60PW-F, J11 XT60PW-F, J12 XT60PW-F, J13 XT60PW-F, J14 1053131302, J15 1053131302, J16 1053131302, J17 1053131302, J18 XT60PW-F, J2 12402012E212A, J3 DEBUG, J4 Conn_02x18_Odd_Even, J5 Conn_02x18_Odd_Even, J6 XT60PW-M, J7 5024940670, J8 1053131303, J9 SM06B-GHS-TB, Q1 DNBT8105-7, Q10 DNBT8105-7, Q11 DNBT8105-7, Q12 DNBT8105-7, Q13 BSS308PE_H6327, Q2 DNBT8105-7, Q3 DNBT8105-7, Q4 DNBT8105-7, Q5 DNBT8105-7, Q6 DNBT8105-7, Q7 DNBT8105-7, Q8 DNBT8105-7, Q9 DNBT8105-7, SW1 KMR223G LFG, SW2 KMR223G LFG, U1 CD74HC4067M, U2 BQ7697202PFBR, U3 W25Q128JVSIQ TR, U4 NCP1117ST33T3G, U5 RP2040, U6 SIC461ED-T1-GE3, U7 ACS72981KLRATR-150B5, X1 ABM8-272-T3

Commit message: feat: schematic pretty much done
Parts:
- added TP1: TestPoint, TestPoint:TestPoint_Pad_D1.5mm, F.Cu at (153.6, 103.1)
- added TP10: TestPoint, TestPoint:TestPoint_Pad_D1.5mm, F.Cu at (139.5, 85.3)
- added TP11: TestPoint, TestPoint:TestPoint_Pad_D1.5mm, F.Cu at (139.5, 88.8)
- added TP12: TestPoint, TestPoint:TestPoint_Pad_D1.5mm, F.Cu at (139.5, 92.4)
- added TP13: TestPoint, TestPoint:TestPoint_Pad_D1.5mm, F.Cu at (143.1, 81.7)
- added TP14: TestPoint, TestPoint:TestPoint_Pad_D1.5mm, F.Cu at (143.1, 85.3)
- added TP15: TestPoint, TestPoint:TestPoint_Pad_D1.5mm, F.Cu at (143.1, 88.8)
- added TP16: TestPoint, TestPoint:TestPoint_Pad_D1.5mm, F.Cu at (158.0, 146.4)
- added TP17: TestPoint, TestPoint:TestPoint_Pad_D1.5mm, F.Cu at (158.0, 150.0)
- added TP18: TestPoint, TestPoint:TestPoint_Pad_D1.5mm, F.Cu at (158.0, 153.5)
- added TP19: TestPoint, TestPoint:TestPoint_Pad_D1.5mm, F.Cu at (102.8, 83.3)
- added TP2: TestPoint, TestPoint:TestPoint_Pad_D1.5mm, F.Cu at (153.6, 106.7)
- added TP20: TestPoint, TestPoint:TestPoint_Pad_D1.5mm, F.Cu at (35.7, 105.1)
- added TP21: TestPoint, TestPoint:TestPoint_Pad_D1.5mm, F.Cu at (102.8, 90.4)
- added TP3: TestPoint, TestPoint:TestPoint_Pad_D1.5mm, F.Cu at (153.6, 110.2)
- added TP4: TestPoint, TestPoint:TestPoint_Pad_D1.5mm, F.Cu at (153.6, 113.8)
- added TP5: TestPoint, TestPoint:TestPoint_Pad_D1.5mm, F.Cu at (136.0, 81.7)
- added TP6: TestPoint, TestPoint:TestPoint_Pad_D1.5mm, F.Cu at (136.0, 85.3)
- added TP7: TestPoint, TestPoint:TestPoint_Pad_D1.5mm, F.Cu at (136.0, 88.8)
- added TP8: TestPoint, TestPoint:TestPoint_Pad_D1.5mm, F.Cu at (136.0, 92.4)
- added TP9: TestPoint, TestPoint:TestPoint_Pad_D1.5mm, F.Cu at (139.5, 81.7)
- C14, C15, C21, C22, C43: value 1u -> 1µ
- C33: value 1µ -> 0.1µ; footprint FixedWing:CAPC1608X90N -> FixedWing:CAP_GCJ-18_MUR
- C36: value 0.1µ -> 1µ; footprint FixedWing:CAP_GCJ-18_MUR -> FixedWing:CAPC1608X90N
- C40: value 220u -> 220µ; moved to B.Cu
- C45: value 4.7u -> 4.7µ
- C51, C52, C53, C54, C55, C56, C57, C58, C59, C60, C61, C62, C63, C64: value 47u -> 47µ
- C65: value 1.5n -> 0.1µ; footprint FixedWing:G-21_MUR -> FixedWing:CAP_GCJ-18_MUR
- C66: value 0.1µ -> 1.5n; footprint FixedWing:CAP_GCJ-18_MUR -> FixedWing:G-21_MUR
- J1, J10, J11, J15, J16, J17: moved to B.Cu
- J12: value XT60PW-F -> 1053131303; footprint FixedWing:XT60PWF -> FixedWing:105313YY03; moved to B.Cu
- J13: value XT60PW-F -> SM06B-GHS-TB; footprint FixedWing:XT60PWF_Pad -> FixedWing:SM06B-GHS-TB; moved to B.Cu
- J14: value 1053131302 -> XT60PW-F; footprint FixedWing:105313YY02 -> FixedWing:XT60PWF_Pad; moved to B.Cu
- J18: value XT60PW-F -> 1053131302; footprint FixedWing:XT60PWF -> FixedWing:105313YY02; moved to B.Cu
- J2: value 12402012E212A -> 1053141210; footprint FixedWing:AMPHENOL_12402012E212A -> FixedWing:CONN_SD-105314-100_10_MOL; moved to B.Cu
- J3: value DEBUG -> 12402012E212A; footprint Connector_PinHeader_2.54mm:PinHeader_1x03_P2.54mm_Vertical -> FixedWing:AMPHENOL_12402012E212A; moved to B.Cu
- J4: value Conn_02x18_Odd_Even -> DEBUG; footprint Connector_PinHeader_2.54mm:PinHeader_2x18_P2.54mm_Vertical -> Connector_PinHeader_2.54mm:PinHeader_1x03_P2.54mm_Vertical; moved to B.Cu
- J5: value Conn_02x18_Odd_Even -> Conn_02x20_Counter_Clockwise; footprint Connector_PinHeader_2.54mm:PinHeader_2x18_P2.54mm_Vertical -> Connector_PinHeader_2.54mm:PinHeader_2x20_P2.54mm_Vertical; moved to B.Cu
- J6: value XT60PW-M -> XT60PW-F; footprint FixedWing:XT60PWM_Pad -> FixedWing:XT60PWF; moved to B.Cu
- J7: value 5024940670 -> XT60PW-M; footprint FixedWing:5024940670 -> FixedWing:XT60PWM_Pad; moved to B.Cu
- J8: value 1053131303 -> XT60PW-F; footprint FixedWing:105313YY03 -> FixedWing:XT60PWF; moved to B.Cu
- J9: value SM06B-GHS-TB -> 5024940670; footprint FixedWing:SM06B-GHS-TB -> FixedWing:5024940670; moved to B.Cu
- NT1: footprint NetTie:NetTie-2_SMD_Pad2.0mm -> NetTie:NetTie-2_SMD_Pad0.5mm
- R100: value 5.6k -> 10k; footprint FixedWing:RESC2012X60N -> FixedWing:KOA_Speer-RK73H2A-0-0-MFG
- R111, R71, R72, R73, R74, R75, R76, R77, R78, R79, R81, R82, R83, R84, R85, R86, R87, R88, R89: footprint FixedWing:RC1206N_YAG -> FixedWing:RES_CRCW_0805_VIS
- moved J13 225.8 mm to (260.2, 63.1), turned to -90 degrees
- moved H4 209.4 mm to (249.1, 154.9)
- moved J12 208.9 mm to (246.4, 109.2), turned to -90 degrees
- moved J11 200.9 mm to (222.0, 148.3)
- moved J9 193.7 mm to (256.5, 50.8), turned to -90 degrees
- moved J14 193.0 mm to (242.6, 90.6), turned to 90 degrees
- moved H2 190.8 mm to (246.4, 33.0)
- moved J18 164.5 mm to (201.6, 150.1), turned to 180 degrees
- moved J8 147.4 mm to (202.1, 39.7), turned to 180 degrees
- moved H6 145.0 mm to (215.9, 78.6)
- moved H8 138.7 mm to (215.9, 86.4)
- moved H5 138.7 mm to (207.9, 78.4)
- moved H7 133.2 mm to (208.3, 86.1)
- moved J3 127.5 mm to (254.0, 124.5), turned to -90 degrees
- moved Q1 114.6 mm to (38.1, 94.0)
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Connections:
- C33 pad 1: GND -> +3V3
- C33 pad 2: +3V3 -> GND
- C34 pad 1: +3V3 -> GND
- C34 pad 2: GND -> +3V3
- C35 pad 1: GND -> +3V3
- C35 pad 2: +3V3 -> GND
- C36 pad 1: +3V3 -> GND
- C36 pad 2: GND -> +3V3
- C65 pad 2: /Battery Stack Monitor/CUR_SENSE -> +5V
- C66 pad 2: +5V -> /Battery Stack Monitor/CUR_SENSE
- D2 pad 2: Net-(J2-VBUS) -> Net-(J3-VBUS)
- J12 pad 1: +BATT -> +5V
- J12 pad 2: /Battery Stack Monitor/GNDCUR -> /External Connections and Sensing/RGB_DOUT
- J13 pad 1: +BATT -> +5V
- J13 pad 2: /Battery Stack Monitor/GNDCUR -> +5V
- J13 pad 3: unconnected-(J13-MH1-Pad3) -> /Battery Stack Monitor/CUR_SENSE
- J13 pad 4: unconnected-(J13-MH2-Pad4) -> Net-(J13-Pad4)
- J14 pad 1: +5V -> +BATT
- J14 pad 2: GND -> /Battery Stack Monitor/GNDCUR
- J15 pad 2: GND -> /Battery Stack Monitor/GNDCUR
- J16 pad 2: GND -> /Battery Stack Monitor/GNDCUR
- J17 pad 2: GND -> /Battery Stack Monitor/GNDCUR
- J18 pad 1: +BATT -> +5V
- J4 pad 1: GND -> /Microcontroller/SWCLK
- J4 pad 2: +3V3 -> GND
- J4 pad 3: GND -> /Microcontroller/SWD
- J5 pad 1: /Microcontroller/GPIO29_ADC3 -> /Battery Stack Monitor/SPI_TX
- J5 pad 10: GND -> /Battery Stack Monitor/RST_SHUT
- J5 pad 11: /Microcontroller/GPIO24 -> /External Connections and Sensing/RGB_DIN
- J5 pad 12: GND -> /Microcontroller/GPIO9
- J5 pad 13: /Microcontroller/GPIO23 -> GND
- J5 pad 14: GND -> /Microcontroller/GPIO10
- J5 pad 15: /Microcontroller/GPIO22 -> /Microcontroller/GPIO11
- J5 pad 16: GND -> /Microcontroller/GPIO12
- J5 pad 17: /Microcontroller/GPIO21 -> /Microcontroller/GPIO13
- J5 pad 19: /Microcontroller/GPIO20 -> /Microcontroller/GPIO14
- J5 pad 2: GND -> /Battery Stack Monitor/SPI_CS
- J5 pad 20: GND -> /Microcontroller/GPIO15
- J5 pad 21: /Microcontroller/GPIO19 -> /Microcontroller/GPIO16
- J5 pad 22: GND -> /Microcontroller/GPIO17
- J5 pad 23: /Microcontroller/GPIO18 -> GND
- J5 pad 24: GND -> /Microcontroller/GPIO18
- J5 pad 25: /Microcontroller/GPIO17 -> /Microcontroller/GPIO19
- J5 pad 26: GND -> /Microcontroller/GPIO20
- J5 pad 27: /Microcontroller/GPIO16 -> /Microcontroller/GPIO21
- J5 pad 29: /Microcontroller/RUN -> /Microcontroller/GPIO22
- J5 pad 3: /Microcontroller/GPIO28_ADC2 -> GND
- J5 pad 30: GND -> /Microcontroller/RUN
- J5 pad 31: /Microcontroller/SWD -> /Microcontroller/GPIO23
- J5 pad 32: GND -> /Microcontroller/GPIO24
- J5 pad 33: /Microcontroller/SWCLK -> GND
- J5 pad 34: GND -> /Microcontroller/GPIO25
- J5 pad 35: GND -> /Microcontroller/GPIO26_ADC0
- J5 pad 36: GND -> /Microcontroller/GPIO27_ADC1
- J5 pad 4: GND -> /Battery Stack Monitor/SPI_SCLK
- J5 pad 5: /Microcontroller/GPIO27_ADC1 -> /Battery Stack Monitor/SPI_RX
- J5 pad 6: GND -> /External Connections and Sensing/PIXDAT
- J5 pad 7: /Microcontroller/GPIO26_ADC0 -> /External Connections and Sensing/PIXCLK
- J5 pad 9: /Microcontroller/GPIO25 -> /Battery Stack Monitor/ALERT
- J6 pad 1: /Battery Stack Monitor/-BATT -> +BATT
- J6 pad 2: Net-(U7-IP+) -> /Battery Stack Monitor/GNDCUR
- J6 pad 3: unconnected-(J6-Pad3) -> GND
- J6 pad 4: unconnected-(J6-Pad4) -> GND
- J7 pad 1: +5V -> /Battery Stack Monitor/-BATT
- J7 pad 2: +5V -> Net-(U7-IP+)
- J7 pad 3: /Microcontroller/GPIO5 -> unconnected-(J7-Pad3)
- J7 pad 4: /Microcontroller/GPIO4 -> unconnected-(J7-Pad4)
- J8 pad 1: +5V -> +BATT
- J8 pad 2: /External Connections and Sensing/RGB_DOUT -> /Battery Stack Monitor/GNDCUR
- J9 pad 3: /Battery Stack Monitor/CUR_SENSE -> /External Connections and Sensing/PIXCLK
- J9 pad 4: Net-(J9-Pad4) -> /External Connections and Sensing/PIXDAT
- LED15 pad 4: /Microcontroller/GPIO8 -> /External Connections and Sensing/RGB_DIN
- NT1 pad 2: /Battery Stack Monitor/-BATT -> /Battery Stack Monitor/GNDCUR
- Q1 pad 1: /Battery Stack Monitor/C0 -> Net-(Q1-B)
- Q13 pad 1: Net-(J2-VBUS) -> Net-(J3-VBUS)
- R100 pad 2: /Microcontroller/~{RESET} -> /Microcontroller/RUN
- R122 pad 2: Net-(J9-Pad4) -> Net-(J13-Pad4)
- R123 pad 1: Net-(J9-Pad4) -> Net-(J13-Pad4)
- R2 pad 2: /Battery Stack Monitor/C0 -> Net-(Q1-B)
- R94 pad 2: /Microcontroller/GPIO7 -> /Battery Stack Monitor/RST_SHUT
- R95 pad 2: Net-(J2-CC1_B) -> Net-(J3-CC1_B)
- R96 pad 2: Net-(J2-CC1_A) -> Net-(J3-CC1_A)
- SW1 pad 1: /Microcontroller/~{RESET} -> /Microcontroller/RUN
- SW1 pad 2: /Microcontroller/~{RESET} -> /Microcontroller/RUN
- U2 pad 21: unconnected-(U2-TS1-Pad21) -> Net-(U2-TS1)
- U2 pad 22: unconnected-(U2-TS2-Pad22) -> Net-(U2-TS2)
- U2 pad 23: unconnected-(U2-TS3-Pad23) -> Net-(U2-TS3)
- U2 pad 25: /Microcontroller/GPIO6 -> /Battery Stack Monitor/ALERT
- U2 pad 26: /Microcontroller/GPIO2 -> /Battery Stack Monitor/SPI_SCLK
- U2 pad 27: /Microcontroller/GPIO0 -> /Battery Stack Monitor/SPI_TX
- U2 pad 28: /Microcontroller/GPIO3 -> /Battery Stack Monitor/SPI_RX
- U2 pad 29: /Microcontroller/GPIO1 -> /Battery Stack Monitor/SPI_CS
- U2 pad 31: unconnected-(U2-DCHG-Pad31) -> Net-(U2-DCHG)
- U2 pad 32: unconnected-(U2-DDSG-Pad32) -> Net-(U2-DDSG)
- U2 pad 33: /Microcontroller/GPIO7 -> /Battery Stack Monitor/RST_SHUT
- U3 pad 4: unconnected-(U3-GND-Pad4) -> GND
- U5 pad 11: /Microcontroller/GPIO8 -> /External Connections and Sensing/RGB_DIN
- U5 pad 2: /Microcontroller/GPIO0 -> /Battery Stack Monitor/SPI_TX
- U5 pad 26: /Microcontroller/~{RESET} -> /Microcontroller/RUN
- U5 pad 3: /Microcontroller/GPIO1 -> /Battery Stack Monitor/SPI_CS
- U5 pad 4: /Microcontroller/GPIO2 -> /Battery Stack Monitor/SPI_SCLK
- U5 pad 5: /Microcontroller/GPIO3 -> /Battery Stack Monitor/SPI_RX
- U5 pad 6: /Microcontroller/GPIO4 -> /External Connections and Sensing/PIXDAT
- U5 pad 7: /Microcontroller/GPIO5 -> /External Connections and Sensing/PIXCLK
- U5 pad 8: /Microcontroller/GPIO6 -> /Battery Stack Monitor/ALERT
- U5 pad 9: /Microcontroller/GPIO7 -> /Battery Stack Monitor/RST_SHUT
- Z1 pad 1: /Battery Stack Monitor/C0 -> Net-(Q1-B)

Commit message: feat: started layout
Parts:
- U7: moved to B.Cu
- moved C16 283.3 mm to (445.0, 121.4)
- moved C19 283.3 mm to (445.0, 124.5)
- moved C2 283.3 mm to (361.9, 90.7)
- moved C23 283.3 mm to (429.0, 106.1)
- moved C24 283.3 mm to (429.0, 109.1)
- moved C25 283.3 mm to (411.1, 90.6)
- moved C29 283.3 mm to (411.1, 93.1)
- moved C3 283.3 mm to (361.9, 93.2)
- moved C30 283.3 mm to (411.1, 95.7)
- moved C32 283.3 mm to (411.1, 98.2)
- moved C33 283.3 mm to (411.1, 100.8)
- moved C34 283.3 mm to (411.1, 103.3)
- moved C4 283.3 mm to (361.9, 95.8)
- moved C40 283.3 mm to (462.5, 154.9)
- moved C44 283.3 mm to (466.7, 162.2)
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Other:
- board outline added: 150 x 100 mm

Commit message: feat: schematic cleanup, continued layout
Parts:
- removed the C66 at (361.7, 124.2)
- removed TP20, TP21: TestPoint, TestPoint:TestPoint_Pad_D1.5mm
- added C65: 10µ, FixedWing:CAP_CL21B106KOQNNNE_SAM, F.Cu at (379.4, 164.8)
- added C68: 0.1µ, FixedWing:CAP_GCJ-18_MUR, F.Cu at (379.2, 159.0)
- added C69: 0.1µ, FixedWing:CAP_GCJ-18_MUR, F.Cu at (379.2, 153.9)
- added C70: 10µ, FixedWing:CAP_CL21B106KOQNNNE_SAM, F.Cu at (379.4, 161.8)
- added C71: 1µ, FixedWing:CAPC1608X90N, F.Cu at (383.3, 153.9)
- added C72: 1µ, FixedWing:CAPC1608X90N, F.Cu at (383.3, 156.3)
- added R124: 100, FixedWing:RESC2012X50N, F.Cu at (369.1, 160.2)
- added R125: 100, FixedWing:RESC2012X50N, F.Cu at (369.1, 166.3)
- added U8: MCP9700AT-E/TT, FixedWing:SOT-23_MC_MCH, F.Cu at (374.8, 160.1)
- added U9: MCP9700AT-E/TT, FixedWing:SOT-23_MC_MCH, F.Cu at (374.8, 155.1)
- R110: value 41.2 -> 41.2k
- R120: value 5.6k -> 8.16k; footprint FixedWing:RESC2012X60N -> FixedWing:RC0805N_YAG
- R121: value 100 -> 475
- R123: value 100k -> 100; footprint FixedWing:RESC2012X60N -> FixedWing:RESC2012X50N
- U7: value ACS72981KLRATR-150B5 -> MCP4726A0T-E/CH; footprint FixedWing:ACS780LLRTR050BT -> FixedWing:SOT-23-6_MC_MCH; moved to F.Cu
- moved U7 365.2 mm to (374.1, 165.0), turned to 0 degrees
- moved Q3 271.6 mm to (105.5, 106.2), turned to 90 degrees
- moved Q9 271.2 mm to (104.0, 55.0), turned to 90 degrees
- moved Q2 270.2 mm to (104.4, 114.5), turned to 90 degrees
- moved Q6 269.8 mm to (104.9, 82.7), turned to 90 degrees
- moved Q8 266.7 mm to (104.0, 65.2), turned to 90 degrees
- moved Q5 266.3 mm to (104.9, 90.7), turned to 90 degrees
- moved Q4 262.1 mm to (105.9, 98.0), turned to 90 degrees
- moved Q7 261.7 mm to (105.0, 74.3), turned to 90 degrees
- moved LED9 259.2 mm to (110.6, 53.0)
- moved LED5 257.8 mm to (110.0, 89.7)
- moved LED2 257.5 mm to (109.6, 114.5)
- moved C9 256.9 mm to (112.0, 57.8), turned to 90 degrees
- moved LED6 256.1 mm to (110.3, 81.7)
- moved C8 255.8 mm to (111.5, 68.0), turned to 90 degrees
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- renumbered C65 to C66, J14 to J13, J15 to J14, J13 to J15
Connections:
- net /Microcontroller/GPIO12 renamed /Microcontroller/DACDAT
- net /Microcontroller/GPIO26_ADC0 renamed /Microcontroller/TEMP_BAL
- net /Microcontroller/GPIO27_ADC1 renamed /Microcontroller/TEMP_CORE
- net /Microcontroller/GPIO9 renamed /Microcontroller/DACCLK
- C2 pad 1: GND -> /Battery Stack Monitor/C1
- C2 pad 2: /Battery Stack Monitor/C1 -> /Battery Stack Monitor/C0
- C67 pad 1: +5V -> GND
- C67 pad 2: GND -> +3.3V
- J1 pad 1: Net-(Q1-E) -> GND
- J10 pad 2: /Battery Stack Monitor/GNDCUR -> GNDPWR
- J10 pad 3: GND -> unconnected-(J10-MH1-Pad3)
- J10 pad 4: GND -> unconnected-(J10-MH2-Pad4)
- J11 pad 2: /Battery Stack Monitor/GNDCUR -> GNDPWR
- J11 pad 3: GND -> unconnected-(J11-MH1-Pad3)
- J11 pad 4: GND -> unconnected-(J11-MH2-Pad4)
- J13 pad 2: /Battery Stack Monitor/GNDCUR -> GNDPWR
- J14 pad 2: /Battery Stack Monitor/GNDCUR -> GNDPWR
- J15 pad 3: /Battery Stack Monitor/CUR_SENSE -> Net-(U7-VOUT)
- J15 pad 4: Net-(J13-Pad4) -> Net-(J15-Pad4)
- J16 pad 2: /Battery Stack Monitor/GNDCUR -> GNDPWR
- J17 pad 2: /Battery Stack Monitor/GNDCUR -> GNDPWR
- J18 pad 2: /Battery Stack Monitor/GNDCUR -> GNDPWR
- J5 pad 6: /External Connections and Sensing/PIXDAT -> /Microcontroller/PIXDAT
- J5 pad 7: /External Connections and Sensing/PIXCLK -> /Microcontroller/PIXCLK
- J6 pad 2: /Battery Stack Monitor/GNDCUR -> GNDPWR
- J6 pad 3: GND -> unconnected-(J6-MH1-Pad3)
- J6 pad 4: GND -> unconnected-(J6-MH2-Pad4)
- J7 pad 2: Net-(U7-IP+) -> +BATT
- J8 pad 2: /Battery Stack Monitor/GNDCUR -> GNDPWR
- J8 pad 3: GND -> unconnected-(J8-MH1-Pad3)
- J8 pad 4: GND -> unconnected-(J8-MH2-Pad4)
- J9 pad 3: /External Connections and Sensing/PIXCLK -> /External Connections and Sensing/PIX_CLK
- J9 pad 4: /External Connections and Sensing/PIXDAT -> /External Connections and Sensing/PIX_DAT
- NT1 pad 2: /Battery Stack Monitor/GNDCUR -> GNDPWR
- Q1 pad 2: Net-(Q1-E) -> GND
- R1 pad 1: Net-(Q1-E) -> GND
- R120 pad 1: GND -> +BATT
- R120 pad 2: Net-(R120-Pad2) -> Net-(J15-Pad4)
- R121 pad 1: Net-(R120-Pad2) -> GND
- R121 pad 2: Net-(R121-Pad2) -> Net-(J15-Pad4)
- R122 pad 1: Net-(R121-Pad2) -> +5V
- R122 pad 2: Net-(J13-Pad4) -> Net-(R122-Pad2)
- R123 pad 1: Net-(J13-Pad4) -> +5V
- R123 pad 2: +BATT -> Net-(R123-Pad2)
- R92 pad 2: /Battery Stack Monitor/GNDCUR -> GNDPWR
- R93 pad 2: /Battery Stack Monitor/GNDCUR -> GNDPWR
- TP19 pad 1: /Battery Stack Monitor/CUR_SENSE -> +BATT
- TP4 pad 1: /Battery Stack Monitor/GNDCUR -> GNDPWR
- U2 pad 30: /Battery Stack Monitor/CUR_SENSE -> unconnected-(U2-DFETOFF-Pad30)
- U5 pad 6: /External Connections and Sensing/PIXDAT -> /Microcontroller/PIXDAT
- U5 pad 7: /External Connections and Sensing/PIXCLK -> /Microcontroller/PIXCLK
- U7 pad 1: +5V -> Net-(U7-VOUT)
- U7 pad 3: /Battery Stack Monitor/CUR_SENSE -> +5V
- U7 pad 4: GND -> /External Connections and Sensing/DAC_DAT
- U7 pad 5: Net-(U7-IP+) -> /External Connections and Sensing/DAC_CLK
- U7 pad 6: +BATT -> +3.3V
- Z1 pad 2: Net-(Q1-E) -> GND

Commit message: feat: placing cell filtering/balancing components
Parts:
- added CR1: USBLC6-2SC6, FixedWing:SOT23-6L_STM, F.Cu at (159.1, -15.0)
- H1, H2, H3, H4, H5, H6, H7, H8: footprint MountingHole:MountingHole_3.2mm_M3_Pad_Via -> MountingHole:MountingHole_3.2mm_M3_ISO14580_Pad
- R92: moved to B.Cu
- U1: value CD74HC4067M -> CD74HC4067; footprint FixedWing:SOIC-24W_7.5x15.4mm_P1.27mm -> FixedWing:DB0024A_N
- moved R92 412.3 mm to (58.0, 76.0)
- moved U2 386.5 mm to (81.2, 108.5), turned to -90 degrees
- moved R66 374.8 mm to (92.5, 81.9)
- moved R64 374.8 mm to (92.5, 77.5)
- moved R65 374.8 mm to (92.5, 80.1)
- moved R68 374.8 mm to (96.3, 74.9)
- moved R70 374.8 mm to (96.3, 80.1)
- moved R69 374.7 mm to (96.3, 78.3)
- moved R63 374.7 mm to (92.5, 75.8)
- moved R67 374.7 mm to (96.3, 73.2)
- moved R89 374.0 mm to (72.5, 95.8)
- moved U1 373.4 mm to (83.2, 83.6)
- moved R88 372.0 mm to (74.5, 99.0)
- moved R87 370.0 mm to (76.5, 95.8)
- moved R79 368.9 mm to (73.0, 92.8), turned to -90 degrees
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Connections:
- net Net-(J3-VBUS) renamed /Microcontroller/VBUS
- J3 pad A6: /Microcontroller/USB_D+ -> Net-(J3-D+_A)
- J3 pad A7: /Microcontroller/USB_D- -> Net-(J3-D-_A)
- J3 pad B6: /Microcontroller/USB_D+ -> Net-(J3-D+_A)
- J3 pad B7: /Microcontroller/USB_D- -> Net-(J3-D-_A)
- R95 pad 1: GND -> Net-(J3-CC1_B)
- R95 pad 2: Net-(J3-CC1_B) -> GND
- R96 pad 1: GND -> Net-(J3-CC1_A)
- R96 pad 2: Net-(J3-CC1_A) -> GND
Routing:
- net Net-(U1-COM): track 0.00 -> 21.5 mm

Commit message: feat: lotta layout
Parts:
- removed the C15 at (136.3, -11.4)
- removed the C21 at (163.2, -23.5)
- removed the C22 at (163.2, -21.0)
- removed the J5 at (84.7, 24.1)
- removed the R118 at (683.4, 190.8)
- added C20: 4.7µ, FixedWing:CAPC2012X145N, B.Cu at (78.0, 114.4)
- added C38: 0.1µ, FixedWing:CAP_GCJ-18_MUR, B.Cu at (118.6, 105.1)
- added C41: 0.1µ, FixedWing:CAP_GCJ-18_MUR, F.Cu at (126.9, 147.8)
- added LED13: LTST-C170KGKT, FixedWing:LED_LTST-C170KGKT_LTO, F.Cu at (120.6, 145.1)
- added R109: 93.1k, FixedWing:RESC2012X60N, F.Cu at (127.0, 145.1)
- added R96: 5.1k, FixedWing:RESC2012X60N, F.Cu at (176.1, 112.3)
- C15: renamed from C16; moved to B.Cu
- C27: renamed from C29; moved to B.Cu
- C28: renamed from C30; moved to B.Cu
- C29: renamed from C31; moved to B.Cu
- C30: renamed from C32; moved to B.Cu
- C31: renamed from C33; moved to B.Cu
- C32: renamed from C34; moved to B.Cu
- C33: renamed from C35; moved to B.Cu
- C34: renamed from C36; moved to B.Cu
- C35: renamed from C37; moved to B.Cu
- C36: renamed from C38; moved to B.Cu
- C37: renamed from C39; moved to B.Cu
- C49: moved to B.Cu
- J4: value DEBUG -> Conn_02x14_Top_Bottom; footprint Connector_PinHeader_2.54mm:PinHeader_1x03_P2.54mm_Vertical -> Connector_PinHeader_2.54mm:PinHeader_2x14_P2.54mm_Vertical; moved to F.Cu
- R116: renamed from R108; value 10k -> 5.1k; footprint FixedWing:KOA_Speer-RK73H2A-0-0-MFG -> FixedWing:RESC2012X60N
- R119: renamed from R117; moved to B.Cu
- R95: value 5.6k -> 5.1k
- R98: renamed from R96; value 5.6k -> 5.1k
- U2: value BQ7697202PFBR -> BQ7697204PFBR
- moved C49 607.5 mm to (116.0, 59.9), turned to -90 degrees
- moved C47 607.4 mm to (115.5, 46.8), turned to -90 degrees
- moved C39 607.2 mm to (107.2, 51.6), turned to -90 degrees
- moved C40 603.1 mm to (119.4, 46.5), turned to -90 degrees
- moved C45 601.7 mm to (120.9, 61.4), turned to 180 degrees
- moved R111 599.0 mm to (124.9, 48.9), turned to 180 degrees
- moved L1 598.3 mm to (110.3, 66.4), turned to -90 degrees
- moved C44 593.2 mm to (126.0, 57.5), turned to 180 degrees
- moved R112 592.2 mm to (122.1, 59.4)
- moved C42 586.7 mm to (129.9, 53.3), turned to -90 degrees
- moved R117 585.7 mm to (126.0, 55.7), turned to 180 degrees
- moved C43 584.7 mm to (124.8, 47.3)
- moved R113 584.1 mm to (124.1, 44.8), turned to -90 degrees
- moved U6 582.9 mm to (117.5, 51.6), turned to -90 degrees
- moved R120 582.8 mm to (125.0, 52.5)
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- renumbered C17 to C16, C18 to C17, C19 to C18, C20 to C19, C23 to C21, C24 to C22, C25 to C23, C26 to C24, C27 to C25, C28 to C26, C40 to C39, C41 to C40, J11 to J10, J12 to J11, J13 to J12, J14 to J13, J15 to J14, J16 to J15, J17 to J16, J18 to J17, J6 to J5, J7 to J6, J8 to J7, J9 to J8, J10 to J9, LED13 to LED14, LED14 to LED15, LED15 to LED16, R99 to R100, R100 to R101, R101 to R102, R102 to R103, R103 to R104, R104 to R105, R105 to R106, R106 to R107, R107 to R108, R109 to R110, R110 to R111, R111 to R112, R112 to R113, R113 to R114, R114 to R115, R115 to R117, R116 to R118, R119 to R120, R120 to R121, R121 to R122, R122 to R123, R123 to R124, R124 to R125, R125 to R126, R98 to R99, SW2 to SW1, SW1 to SW2, TP8 to TP10, TP9 to TP8, TP10 to TP9
Connections:
- J4 pad 1: /Microcontroller/SWCLK -> +5V
- J4 pad 2: GND -> /Microcontroller/GPIO12
- J4 pad 3: /Microcontroller/SWD -> /Microcontroller/GPIO13
- LED15 pad 1: GNDA -> GND
- LED15 pad 2: Net-(LED14-A) (its old number) -> Net-(LED15-A)
- R116 pad 1: Net-(U6-VDD) -> Net-(LED15-A)
- R116 pad 2: Net-(LED14-A) (its old number) -> +5V
- R95 pad 1: Net-(J3-CC1_B) -> GND
- R95 pad 2: GND -> Net-(J3-CC1_B)
- R98 pad 1: Net-(J3-CC1_A) -> +3V3
- R98 pad 2: GND -> Net-(LED13-A)
- TP17 pad 1: Net-(LED14-A) (its old number) -> /5V Regulator/PGOOD
- U5 pad 11: /External Connections and Sensing/RGB_DIN -> /Microcontroller/PIXDAT
- U5 pad 12: /Microcontroller/DACCLK -> /Microcontroller/PIXCLK
- U5 pad 13: /Microcontroller/GPIO10 -> /Microcontroller/DACDAT
- U5 pad 14: /Microcontroller/GPIO11 -> /Microcontroller/DACCLK
- U5 pad 15: /Microcontroller/DACDAT -> /Microcontroller/GPIO12
- U5 pad 6: /Microcontroller/PIXDAT -> /Battery Stack Monitor/ALERT
- U5 pad 7: /Microcontroller/PIXCLK -> /Battery Stack Monitor/RST_SHUT
- U5 pad 8: /Battery Stack Monitor/ALERT -> /External Connections and Sensing/RGB_DIN
- U5 pad 9: /Battery Stack Monitor/RST_SHUT -> /Microcontroller/PGOOD
- U6 pad 2: Net-(LED14-A) (its old number) -> /5V Regulator/PGOOD
Routing:
- net /Battery Stack Monitor/C11: track 0.00 -> 69.8 mm
- net /Battery Stack Monitor/C10: track 0.00 -> 62.1 mm
- net Net-(J1-Pad13): track 0.00 -> 56.0 mm
- net /Battery Stack Monitor/C12: track 0.00 -> 55.9 mm
- net /Battery Stack Monitor/C9: track 0.00 -> 52.1 mm
- net /Battery Stack Monitor/C8: track 0.00 -> 44.0 mm
- net /Battery Stack Monitor/C7: track 0.00 -> 38.3 mm
- net /Battery Stack Monitor/C6: track 0.00 -> 30.8 mm
- net /Battery Stack Monitor/C5: track 0.00 -> 25.6 mm
- net /Battery Stack Monitor/C0: track 0.00 -> 24.3 mm
- net Net-(U1-COM): track 21.5 -> 0.00 mm
- net /Battery Stack Monitor/C4: track 0.00 -> 20.7 mm
- net /Battery Stack Monitor/C2: track 0.00 -> 19.4 mm
- net /Battery Stack Monitor/C3: track 0.00 -> 17.7 mm
- net /Battery Stack Monitor/C1: track 0.00 -> 17.4 mm
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