File: bms-kicad-project/bms-board.kicad_pcb (KiCad board)
At the start: 4 copper layers, 150 x 100 mm, 301 parts, among them J1 S13B-XH-A, J10 XT60PW-F, J11 1053131303, J12 XT60PW-F, J13 1053131302, J14 SM06B-GHS-TB, J15 1053131302, J16 1053131302, J17 1053131302, J2 1053141210, J3 12402012E212A, J4 Conn_02x14_Top_Bottom, J5 XT60PW-F, J6 XT60PW-M, J7 XT60PW-F, J8 5024940670, J9 XT60PW-F, Q1 DNBT8105-7, Q10 DNBT8105-7, Q11 DNBT8105-7, Q12 DNBT8105-7, Q13 BSS308PE_H6327, Q2 DNBT8105-7, Q3 DNBT8105-7, Q4 DNBT8105-7, Q5 DNBT8105-7, Q6 DNBT8105-7, Q7 DNBT8105-7, Q8 DNBT8105-7, Q9 DNBT8105-7, SW1 KMR223G LFG, SW2 KMR223G LFG, U1 CD74HC4067, U2 BQ7697204PFBR, U3 W25Q128JVSIQ TR, U4 NCP1117ST33T3G, U5 RP2040, U6 SIC461ED-T1-GE3, U7 MCP4726A0T-E/CH, U8 MCP9700AT-E/TT, U9 MCP9700AT-E/TT, X1 ABM8-272-T3

Commit message: feat: post-design review clarity
Parts:
- added BB1: Busbar, FixedWing:BUSBAR_LONG, F.Cu at (41.5, 158.3)
- added BB2: Busbar, FixedWing:BUSBAR_SHORT, F.Cu at (41.5, 163.6)
- added C14: 0.1µ, FixedWing:CAP_GCJ-18_MUR, F.Cu at (56.5, 193.0)
- added C22: 3.9n, FixedWing:G-21_MUR, F.Cu at (56.6, 175.7)
- added C23: 3.9n, FixedWing:G-21_MUR, F.Cu at (56.6, 178.6)
- added C24: 3.9n, FixedWing:G-21_MUR, F.Cu at (56.6, 181.5)
- added C25: 3.9n, FixedWing:G-21_MUR, F.Cu at (56.6, 184.4)
- added C26: 3.9n, FixedWing:G-21_MUR, F.Cu at (56.6, 187.3)
- added C27: 3.9n, FixedWing:G-21_MUR, F.Cu at (56.6, 190.3)
- added CR2: USBLC6-2SC6, FixedWing:SOT23-6L_STM, B.Cu at (166.5, 99.1)
- added CR3: USBLC6-2SC6, FixedWing:SOT23-6L_STM, B.Cu at (172.0, 59.0)
- added R120: 10k, FixedWing:KOA_Speer-RK73H2A-0-0-MFG, F.Cu at (65.8, 184.7)
- added R122: 10k, FixedWing:KOA_Speer-RK73H2A-0-0-MFG, F.Cu at (65.8, 187.3)
- added R123: 10k, FixedWing:KOA_Speer-RK73H2A-0-0-MFG, F.Cu at (65.8, 189.9)
- added R124: 8.16k, FixedWing:RC0805N_YAG, F.Cu at (69.8, 187.9)
- added R125: 475, FixedWing:RESC2012X50N, F.Cu at (69.9, 184.9)
- added R126: 10k, FixedWing:KOA_Speer-RK73H2A-0-0-MFG, F.Cu at (129.3, 164.2)
- added R127: 10k, FixedWing:KOA_Speer-RK73H2A-0-0-MFG, F.Cu at (129.3, 166.8)
- added TP1: ~, TestPoint:TestPoint_Pad_D1.0mm, F.Cu at (60.3, 175.8)
- added TP11: ~, TestPoint:TestPoint_Pad_D1.0mm, F.Cu at (82.6, 175.8)
- added TP2: ~, TestPoint:TestPoint_Pad_D1.0mm, F.Cu at (60.3, 178.8)
- added TP21: ~, TestPoint:TestPoint_Pad_D1.0mm, F.Cu at (65.4, 175.8)
- added TP25: ~, TestPoint:TestPoint_Pad_D1.0mm, F.Cu at (65.4, 178.8)
- added TP26: ~, TestPoint:TestPoint_Pad_D1.0mm, F.Cu at (65.4, 181.9)
- added TP27: ~, TestPoint:TestPoint_Pad_D1.0mm, F.Cu at (68.4, 175.8)
- added TP28: ~, TestPoint:TestPoint_Pad_D1.0mm, F.Cu at (68.4, 178.8)
- added TP29: ~, TestPoint:TestPoint_Pad_D1.0mm, F.Cu at (68.4, 181.9)
- added TP30: ~, TestPoint:TestPoint_Pad_D1.0mm, F.Cu at (71.5, 175.8)
- added TP31: ~, TestPoint:TestPoint_Pad_D1.0mm, F.Cu at (71.5, 178.8)
- added TP32: ~, TestPoint:TestPoint_Pad_D1.0mm, F.Cu at (71.5, 181.9)
- added TP33: ~, TestPoint:TestPoint_Pad_D1.0mm, F.Cu at (74.5, 175.8)
- added TP34: ~, TestPoint:TestPoint_Pad_D1.0mm, F.Cu at (74.5, 178.8)
- added TP35: ~, TestPoint:TestPoint_Pad_D1.0mm, F.Cu at (74.5, 181.9)
- added TP36: ~, TestPoint:TestPoint_Pad_D1.0mm, F.Cu at (77.6, 175.8)
- added TP37: ~, TestPoint:TestPoint_Pad_D1.0mm, F.Cu at (77.6, 178.8)
- added TP38: ~, TestPoint:TestPoint_Pad_D1.0mm, F.Cu at (77.6, 181.9)
- added TP40: ~, TestPoint:TestPoint_Pad_D1.0mm, F.Cu at (129.0, 169.6)
- added TP6: ~, TestPoint:TestPoint_Pad_D1.0mm, F.Cu at (60.3, 181.9)
- added TP7: ~, TestPoint:TestPoint_Pad_D1.0mm, F.Cu at (60.3, 184.9)
- CR1: moved to B.Cu
- J2: value 1053141210 -> 1053141308; footprint FixedWing:CONN_SD-105314-100_10_MOL -> FixedWing:CONN_SD-105314-100_08_MOL; moved to F.Cu
- TP10: renamed from TP17; value TestPoint -> ~; footprint TestPoint:TestPoint_Pad_D1.5mm -> TestPoint:TestPoint_Pad_D1.0mm
- TP12: renamed from TP18; value TestPoint -> ~; footprint TestPoint:TestPoint_Pad_D1.5mm -> TestPoint:TestPoint_Pad_D1.0mm
- TP13: renamed from TP5; value TestPoint -> ~; footprint TestPoint:TestPoint_Pad_D1.5mm -> TestPoint:TestPoint_Pad_D1.0mm
- TP14: renamed from TP6; value TestPoint -> ~; footprint TestPoint:TestPoint_Pad_D1.5mm -> TestPoint:TestPoint_Pad_D1.0mm
- TP15: renamed from TP7; value TestPoint -> ~; footprint TestPoint:TestPoint_Pad_D1.5mm -> TestPoint:TestPoint_Pad_D1.0mm
- TP16: renamed from TP8; value TestPoint -> ~; footprint TestPoint:TestPoint_Pad_D1.5mm -> TestPoint:TestPoint_Pad_D1.0mm
- TP17: renamed from TP9; value TestPoint -> ~; footprint TestPoint:TestPoint_Pad_D1.5mm -> TestPoint:TestPoint_Pad_D1.0mm
- TP18: renamed from TP10; value TestPoint -> ~; footprint TestPoint:TestPoint_Pad_D1.5mm -> TestPoint:TestPoint_Pad_D1.0mm
- TP19: renamed from TP11; value TestPoint -> ~; footprint TestPoint:TestPoint_Pad_D1.5mm -> TestPoint:TestPoint_Pad_D1.0mm
- TP20: renamed from TP12; value TestPoint -> ~; footprint TestPoint:TestPoint_Pad_D1.5mm -> TestPoint:TestPoint_Pad_D1.0mm
- TP22: renamed from TP13; value TestPoint -> ~; footprint TestPoint:TestPoint_Pad_D1.5mm -> TestPoint:TestPoint_Pad_D1.0mm
- TP23: renamed from TP14; value TestPoint -> ~; footprint TestPoint:TestPoint_Pad_D1.5mm -> TestPoint:TestPoint_Pad_D1.0mm
- TP24: renamed from TP15; value TestPoint -> ~; footprint TestPoint:TestPoint_Pad_D1.5mm -> TestPoint:TestPoint_Pad_D1.0mm
- TP3: renamed from TP1; value TestPoint -> ~; footprint TestPoint:TestPoint_Pad_D1.5mm -> TestPoint:TestPoint_Pad_D1.0mm
- TP39: renamed from TP19; value TestPoint -> ~; footprint TestPoint:TestPoint_Pad_D1.5mm -> TestPoint:TestPoint_Pad_D1.0mm
- TP4: renamed from TP2; value TestPoint -> ~; footprint TestPoint:TestPoint_Pad_D1.5mm -> TestPoint:TestPoint_Pad_D1.0mm
- TP5: renamed from TP3; value TestPoint -> ~; footprint TestPoint:TestPoint_Pad_D1.5mm -> TestPoint:TestPoint_Pad_D1.0mm
- TP8: renamed from TP4; value TestPoint -> ~; footprint TestPoint:TestPoint_Pad_D1.5mm -> TestPoint:TestPoint_Pad_D1.0mm
- TP9: renamed from TP16; value TestPoint -> ~; footprint TestPoint:TestPoint_Pad_D1.5mm -> TestPoint:TestPoint_Pad_D1.0mm
- moved CR1 27.3 mm to (168.9, 113.7)
- moved J2 3.82 mm to (42.0, 109.7), turned to -90 degrees
- moved R112 1.30 mm to (176.1, 111.0)
- moved R111 0.90 mm to (176.2, 116.0)
- renumbered C14 to C15, C15 to C16, C16 to C17, C17 to C18, C18 to C19, C19 to C20, C20 to C21, C39 to C28, C40 to C29, C41 to C30, C42 to C31, C43 to C32, C44 to C33, C45 to C34, C46 to C35, C47 to C36, C48 to C37, C49 to C38, C50 to C39, C51 to C40, C52 to C41, C53 to C42, C54 to C43, C55 to C44, C56 to C45, C57 to C46, C58 to C47, C59 to C48, C60 to C49, C61 to C50, C62 to C51, C63 to C52, C64 to C53, C21 to C54, C22 to C55, C23 to C56, C24 to C57, C25 to C58, C26 to C59, C27 to C60, C28 to C61, C29 to C62, C30 to C63, C31 to C64, C32 to C65, C33 to C66, C34 to C67, C35 to C68, C36 to C69, C37 to C70, C38 to C71, C66 to C72, C65 to C73, C67 to C74, C68 to C75, C69 to C76, C70 to C77, C71 to C78, C72 to C79, J11 to J10, J12 to J11, J8 to J12, J15 to J14, J16 to J15, J17 to J16, J14 to J17, J9 to J8, J10 to J9, LED15 to LED13, LED13 to LED14, LED14 to LED15, R110 to R100, R111 to R101, R112 to R102, R113 to R103, R114 to R104, R115 to R105, R116 to R106, R117 to R107, R118 to R108, R119 to R109, R120 to R110, R95 to R111, R96 to R112, R97 to R113, R98 to R114, R99 to R115, R100 to R116, R101 to R117, R102 to R118, R103 to R119, R104 to R121, R121 to R128, R122 to R129, R123 to R130, R124 to R131, R125 to R132, R126 to R133, R105 to R95, R106 to R96, R107 to R97, R108 to R98, R109 to R99, U6 to U3, U3 to U4, U4 to U5, U5 to U6
Connections:
- net Net-(U2-TS1) renamed /Battery Stack Monitor/THERM1
- net Net-(U2-TS2) renamed /Battery Stack Monitor/THERM2
- net Net-(U2-TS3) renamed /Battery Stack Monitor/THERM3
- C32 pad 1: Net-(U6-VDD) -> Net-(U3-VDD)
- C73 pad 2: +3.3V -> +3V3
- C74 pad 2: +3.3V -> +3V3
- CR1 pad 1: Net-(J3-D+_A) -> Net-(J3-D-_A)
- CR1 pad 3: Net-(J3-D-_A) -> Net-(J3-D+_A)
- CR1 pad 4: /Microcontroller/USB_D- -> /Microcontroller/USB_D+
- CR1 pad 6: /Microcontroller/USB_D+ -> /Microcontroller/USB_D-
- J12 pad 3: /External Connections and Sensing/PIX_CLK -> Net-(CR2-Pad1)
- J12 pad 4: /External Connections and Sensing/PIX_DAT -> Net-(CR2-Pad3)
- J17 pad 3: Net-(U7-VOUT) -> Net-(CR3-Pad1)
- J17 pad 4: Net-(J14-Pad4) -> Net-(CR3-Pad3)
- J2 pad 4: Net-(U2-DCHG) -> /Battery Stack Monitor/THERM4
- J2 pad 5: Net-(U2-DDSG) -> /Battery Stack Monitor/THERM5
- J2 pad 6: GND -> /Battery Stack Monitor/THERM6
- J4 pad 15: +3.3V -> +3V3
- J4 pad 21: +3.3V -> +3V3
- J4 pad 27: +3.3V -> +3V3
- R102 pad 1: Net-(U6-VDD) -> Net-(U3-VDD)
- R128 pad 2: Net-(J14-Pad4) -> Net-(CR3-Pad4)
- R129 pad 2: Net-(J14-Pad4) -> Net-(CR3-Pad4)
- R99 pad 1: Net-(U6-VDD) -> /5V Regulator/PGOOD
- R99 pad 2: /5V Regulator/PGOOD -> +3V3
- U2 pad 30: unconnected-(U2-DFETOFF-Pad30) -> /Battery Stack Monitor/THERM4
- U2 pad 31: Net-(U2-DCHG) -> /Battery Stack Monitor/THERM5
- U2 pad 32: Net-(U2-DDSG) -> /Battery Stack Monitor/THERM6
- U3 pad 26: Net-(U6-VDD) -> Net-(U3-VDD)
- U6 pad 11: /Microcontroller/PIXDAT -> /External Connections and Sensing/PIX_DAT
- U6 pad 12: /Microcontroller/PIXCLK -> /External Connections and Sensing/PIX_CLK
- U6 pad 13: /Microcontroller/DACDAT -> /External Connections and Sensing/DAC_DAT
- U6 pad 14: /Microcontroller/DACCLK -> /External Connections and Sensing/DAC_CLK
- U6 pad 38: /Microcontroller/TEMP_BAL -> /External Connections and Sensing/TEMP_BAL
- U6 pad 39: /Microcontroller/TEMP_CORE -> /External Connections and Sensing/TEMP_CORE
- U6 pad 9: /Microcontroller/PGOOD -> /5V Regulator/PGOOD
- U7 pad 6: +3.3V -> +3V3

Commit message: feat: I am so tired. 4-layer layout almost done
Parts:
- removed H5, H6, H7, H8: MountingHole_Pad, MountingHole:MountingHole_3.2mm_M3_ISO14580_Pad
- removed NT1: NetTie_2, NetTie:NetTie-2_SMD_Pad0.5mm
- removed NT2: NetTie_3, NetTie:NetTie-3_SMD_Pad2.0mm
- removed the TP1 at (60.3, 175.8)
- removed the TP11 at (82.6, 175.8)
- removed the TP14 at (150.4, 159.9)
- removed the TP15 at (150.4, 163.4)
- removed the TP16 at (153.9, 156.3)
- removed the TP19 at (153.9, 163.4)
- removed the TP20 at (153.9, 167.0)
- removed the TP8 at (60.3, 5.60)
- added C29: 1µ, FixedWing:CAP_CL31_SAM, F.Cu at (102.4, 41.6)
- added C30: 1µ, FixedWing:CAP_CL31_SAM, F.Cu at (104.8, 41.6)
- added C31: 1µ, FixedWing:CAP_CL31_SAM, F.Cu at (107.2, 41.6)
- added C32: 100p, FixedWing:CAPC220145_88N_KEM, F.Cu at (109.6, 41.5)
- added C58: 47µ, FixedWing:G-32_MUR, F.Cu at (132.8, 37.6)
- added C77: 0.1µ, FixedWing:CAP_GCJ-18_MUR, F.Cu at (134.6, 97.6)
- added C78: 1µ, FixedWing:CAPC1608X90N, F.Cu at (134.3, 90.1)
- added C79: 0.1µ, FixedWing:CAP_GCJ-18_MUR, F.Cu at (133.6, 99.3)
- added C80: 1µ, FixedWing:CAPC1608X90N, F.Cu at (133.6, 93.6)
- added MP1: M3 x 15mm, FixedWing:WA-SMSI_9774150360, B.Cu at (94.0, 64.8)
- added MP2: M3 x 15mm, FixedWing:WA-SMSI_9774150360, B.Cu at (124.5, 64.8)
- added MP3: M3 x 15mm, FixedWing:WA-SMSI_9774150360, B.Cu at (94.0, 95.3)
- added MP4: M3 x 15mm, FixedWing:WA-SMSI_9774150360, B.Cu at (124.5, 95.3)
- added R128: 5.1k, FixedWing:RESC2012X60N, F.Cu at (198.8, 44.5)
- added R129: 5.1k, FixedWing:RESC2012X60N, F.Cu at (198.8, 47.4)
- added TP6: 5261, FixedWing:KEYSTONE_5261, F.Cu at (49.0, 2.95)
- BB1, BB2, J2: moved to B.Cu
- C16, C21: moved to F.Cu
- C49: renamed from C45; moved to B.Cu
- C50: renamed from C46; moved to B.Cu
- C51: renamed from C47; moved to B.Cu
- C53: renamed from C49; moved to B.Cu
- C54: renamed from C50; moved to B.Cu
- C55: renamed from C51; moved to B.Cu
- C56: renamed from C52; moved to B.Cu
- C57: renamed from C53; moved to B.Cu
- C65: renamed from C60; moved to F.Cu
- C67: renamed from C62; moved to F.Cu
- C72: renamed from C67; moved to F.Cu
- C73: renamed from C68; moved to F.Cu
- C74: renamed from C69; moved to F.Cu
- C75: renamed from C70; moved to F.Cu
- C76: renamed from C71; moved to F.Cu
- R126, R127: value 10k -> 5.1k; footprint FixedWing:KOA_Speer-RK73H2A-0-0-MFG -> FixedWing:RESC2012X60N
- TP17, TP2, TP5, TP7: value ~ -> 5261; footprint TestPoint:TestPoint_Pad_D1.0mm -> FixedWing:KEYSTONE_5261
- moved LED16 404.8 mm to (147.5, 49.3), turned to 180 degrees
- moved C81 391.0 mm to (161.6, 47.7), turned to -90 degrees
- moved C82 390.9 mm to (148.2, 58.0), turned to 90 degrees
- moved C83 387.7 mm to (150.4, 57.8), turned to 90 degrees
- moved C85 383.6 mm to (154.3, 58.9)
- moved R130 382.3 mm to (156.4, 64.4), turned to 90 degrees
- moved C84 381.4 mm to (157.2, 56.0), turned to 90 degrees
- moved U7 380.3 mm to (153.8, 55.9), turned to 180 degrees
- moved C86 379.6 mm to (159.4, 55.9), turned to 90 degrees
- moved R131 372.1 mm to (155.4, 61.2)
- moved C88 362.0 mm to (179.6, 66.2)
- moved C87 359.7 mm to (181.1, 80.2)
- moved U9 349.3 mm to (183.9, 63.6)
- moved R133 347.9 mm to (180.7, 59.6), turned to -90 degrees
- moved R135 347.8 mm to (180.7, 63.4), turned to -90 degrees
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- renumbered C29 to C33, C30 to C34, C31 to C35, C32 to C36, C33 to C37, C34 to C38, C35 to C39, C36 to C40, C37 to C41, C38 to C42, C39 to C43, C40 to C44, C41 to C45, C42 to C46, C43 to C47, C44 to C48, C48 to C52, C54 to C59, C55 to C60, C56 to C61, C57 to C62, C58 to C63, C59 to C64, C61 to C66, C63 to C68, C64 to C69, C65 to C70, C66 to C71, C72 to C81, C73 to C82, C74 to C83, C75 to C84, C76 to C85, C77 to C86, C78 to C87, C79 to C88, R128 to R130, R129 to R131, R130 to R132, R131 to R133, R132 to R134, R133 to R135, TP3 to TP1, TP12 to TP10, TP13 to TP11, TP18 to TP12, TP21 to TP13, TP22 to TP14, TP23 to TP15, TP24 to TP16, TP25 to TP18, TP26 to TP19, TP27 to TP20, TP28 to TP21, TP29 to TP22, TP30 to TP23, TP31 to TP24, TP32 to TP25, TP33 to TP26, TP34 to TP27, TP35 to TP28, TP36 to TP29, TP4 to TP3, TP37 to TP30, TP38 to TP31, TP39 to TP32, TP40 to TP33, TP6 to TP4, TP9 to TP8, TP10 to TP9
Connections:
- BB2 pad 1: GNDPWR -> GND
- C28 pad 2: GNDPWR -> GND
- C33 pad 1: GNDPWR -> GND
- C34 pad 1: GNDPWR -> GND
- C35 pad 1: GNDA -> GND
- C36 pad 2: GNDA -> GND
- C37 pad 1: GNDA -> GND
- C38 pad 1: GNDPWR -> GND
- C42 pad 2: GNDPWR -> GND
- C43 pad 1: GNDPWR -> GND
- C44 pad 1: GNDPWR -> GND
- C45 pad 1: GNDPWR -> GND
- C46 pad 1: GNDPWR -> GND
- C47 pad 1: GNDPWR -> GND
- C48 pad 1: GNDPWR -> GND
- C49 pad 1: GNDPWR -> GND
- C50 pad 1: GNDPWR -> GND
- C51 pad 1: GNDPWR -> GND
- C52 pad 1: GNDPWR -> GND
- C53 pad 1: GNDPWR -> GND
- C54 pad 1: GNDPWR -> GND
- C55 pad 1: GNDPWR -> GND
- C56 pad 1: GNDPWR -> GND
- C57 pad 1: GNDPWR -> GND
- CR1 pad 1: Net-(J3-D-_A) -> Net-(J3-D+_A)
- CR1 pad 3: Net-(J3-D+_A) -> Net-(J3-D-_A)
- CR1 pad 4: /Microcontroller/USB_D+ -> /Microcontroller/USB_D-
- CR1 pad 6: /Microcontroller/USB_D- -> /Microcontroller/USB_D+
- J11 pad 2: GNDPWR -> GND
- J13 pad 2: GNDPWR -> GND
- J14 pad 2: GNDPWR -> GND
- J15 pad 2: GNDPWR -> GND
- J16 pad 2: GNDPWR -> GND
- J4 pad 10: /Microcontroller/GPIO19 -> /Microcontroller/GPIO15
- J4 pad 11: +5V -> /Microcontroller/SWCLK
- J4 pad 12: /Microcontroller/GPIO20 -> /Microcontroller/SWD
- J4 pad 13: /Microcontroller/GPIO21 -> /Microcontroller/GPIO16
- J4 pad 14: GND -> /Microcontroller/GPIO17
- J4 pad 15: +3V3 -> GND
- J4 pad 16: /Microcontroller/GPIO22 -> GND
- J4 pad 17: /Microcontroller/GPIO23 -> /Microcontroller/GPIO18
- J4 pad 18: GND -> /Microcontroller/GPIO19
- J4 pad 19: /Microcontroller/GPIO24 -> /Microcontroller/GPIO20
- J4 pad 2: /Microcontroller/GPIO12 -> +3V3
- J4 pad 20: /Microcontroller/GPIO25 -> /Microcontroller/GPIO21
- J4 pad 21: +3V3 -> /Microcontroller/GPIO22
- J4 pad 22: /Microcontroller/GPIO28_ADC2 -> /Microcontroller/GPIO23
- J4 pad 23: /Microcontroller/GPIO29_ADC3 -> /Microcontroller/GPIO24
- J4 pad 24: GND -> /Microcontroller/GPIO25
- J4 pad 25: /Microcontroller/SWCLK -> /Microcontroller/GPIO26_ADC0
- J4 pad 26: /Microcontroller/SWD -> GND
- J4 pad 27: +3V3 -> GND
- J4 pad 3: /Microcontroller/GPIO13 -> +5V
- J4 pad 4: /Microcontroller/GPIO14 -> +3V3
- J4 pad 5: /Microcontroller/GPIO15 -> GND
- J4 pad 7: /Microcontroller/GPIO16 -> /Microcontroller/GPIO12
- J4 pad 8: /Microcontroller/GPIO17 -> /Microcontroller/GPIO13
- J4 pad 9: /Microcontroller/GPIO18 -> /Microcontroller/GPIO14
- J5 pad 2: GNDPWR -> GND
- J7 pad 2: GNDPWR -> GND
- J8 pad 2: GNDPWR -> GND
- J9 pad 2: GNDPWR -> GND
- R100 pad 1: GNDA -> GND
- R101 pad 1: GNDA -> GND
- R104 pad 1: GNDA -> GND
- R107 pad 1: GNDA -> GND
- R122 pad 1: /Microcontroller/GPIO28_ADC2 -> /Microcontroller/GPIO27_ADC1
- R123 pad 2: /Microcontroller/GPIO28_ADC2 -> /Microcontroller/GPIO27_ADC1
- R124 pad 2: /Microcontroller/GPIO29_ADC3 -> /Microcontroller/GPIO28_ADC2
- R125 pad 2: /Microcontroller/GPIO29_ADC3 -> /Microcontroller/GPIO28_ADC2
- R126 pad 1: /External Connections and Sensing/DAC_DAT -> /External Connections and Sensing/PIX_CLK
- R127 pad 1: /External Connections and Sensing/DAC_CLK -> /External Connections and Sensing/PIX_DAT
- R92 pad 2: GNDPWR -> GND
- R93 pad 2: GNDPWR -> GND
- R97 pad 1: GNDPWR -> GND
- TP30 pad 1: /External Connections and Sensing/TEMP_BAL -> /External Connections and Sensing/TEMP_ESC
- U3 pad 10: GNDPWR -> GND
- U3 pad 11: GNDPWR -> GND
- U3 pad 17: GNDPWR -> GND
- U3 pad 23: GNDA -> GND
- U3 pad 28: GNDA -> GND
- U3 pad 30.1: GNDPWR -> GND
- U3 pad 30.2: GNDPWR -> GND
- U3 pad 9: GNDPWR -> GND
- U6 pad 38: /External Connections and Sensing/TEMP_BAL -> /Microcontroller/GPIO26_ADC0
- U6 pad 39: /External Connections and Sensing/TEMP_CORE -> /Microcontroller/GPIO27_ADC1
- U6 pad 41: /Microcontroller/GPIO29_ADC3 -> /External Connections and Sensing/TEMP_CORE
- U8 pad 2: /External Connections and Sensing/TEMP_BAL -> /External Connections and Sensing/TEMP_ESC
Routing:
- net GND: track 0.00 -> 131.7 mm, vias 0 -> 142
- net +5V: track 0.00 -> 123.4 mm, vias 0 -> 110
- net /5V Regulator/PGOOD: track 0.00 -> 116.5 mm, vias 0 -> 2
- net +3V3: track 0.00 -> 99.9 mm, vias 0 -> 42
- net Net-(Q12-E): track 0.00 -> 99.6 mm
- net /External Connections and Sensing/PIX_CLK: track 0.00 -> 94.9 mm, vias 0 -> 3
- net /External Connections and Sensing/PIX_DAT: track 0.00 -> 92.7 mm, vias 0 -> 3
- net /External Connections and Sensing/DAC_DAT: track 0.00 -> 85.9 mm, vias 0 -> 2
- net /External Connections and Sensing/DAC_CLK: track 0.00 -> 82.7 mm, vias 0 -> 2
- net Net-(Q11-E): track 0.00 -> 81.8 mm
- net /External Connections and Sensing/RGB_DIN: track 0.00 -> 80.0 mm, vias 0 -> 2
- net Net-(Q10-E): track 0.00 -> 71.0 mm
- net Net-(Q2-E): track 0.00 -> 67.9 mm
- net /Battery Stack Monitor/THERM6: track 0.00 -> 62.4 mm
- net Net-(Q9-E): track 0.00 -> 61.5 mm
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- added copper zone on F.Cu, net +1V1
- added copper zone on B.Cu, net +3V3
- added copper zone on F.Cu, net +3V3
- added copper zone on B.Cu, net +5V
- added copper zone on F.Cu, net +5V
- added copper zone on B.Cu, net +BATT
- added copper zone on F.Cu, net +BATT
- added copper zone on In2.Cu, net +BATT
- added copper zone on B.Cu, net /Battery Stack Monitor/-BATT
- added copper zone on F.Cu, net /Battery Stack Monitor/-BATT
- added copper zone on In2.Cu, net /Battery Stack Monitor/-BATT
- added copper zone on B.Cu, net GND
- added copper zone on F.Cu, net GND
- added copper zone on In2.Cu, net GND
- added copper zone on F.Cu, net Net-(U3-SW)
Other:
- board size 150 x 100 mm -> 140 x 100 mm
