File: bms-kicad-project/CellFilteringAndBalancing.kicad_sch (KiCad schematic)
At the start: 111 parts, among them J18 S13B-XH-A, Q15 DNBT8105-7, Q16 DNBT8105-7, Q17 DNBT8105-7, Q18 DNBT8105-7, Q19 DNBT8105-7, Q20 DNBT8105-7, Q21 DNBT8105-7, Q22 DNBT8105-7, Q23 DNBT8105-7, Q24 DNBT8105-7, Q25 DNBT8105-7, Q26 DNBT8105-7

Commit message: feat: don't even know what I changed, just zoned out for several hours. Made PCB r/a mount XT-60s and solder pads into a 2-for-1 deal
Parts:
- R13: renamed from R115; footprint RES_R1632_ROM -> FixedWing:RES_R1632_ROM
- R14: renamed from R60; footprint RES_R1632_ROM -> FixedWing:RES_R1632_ROM
- R18: renamed from R116; footprint RES_R1632_ROM -> FixedWing:RES_R1632_ROM
- R19: renamed from R61; footprint RES_R1632_ROM -> FixedWing:RES_R1632_ROM
- R23: renamed from R117; footprint RES_R1632_ROM -> FixedWing:RES_R1632_ROM
- R24: renamed from R62; footprint RES_R1632_ROM -> FixedWing:RES_R1632_ROM
- R28: renamed from R118; footprint RES_R1632_ROM -> FixedWing:RES_R1632_ROM
- R29: renamed from R63; footprint RES_R1632_ROM -> FixedWing:RES_R1632_ROM
- R3: renamed from R112; footprint RES_R1632_ROM -> FixedWing:RES_R1632_ROM
- R33: renamed from R113; footprint RES_R1632_ROM -> FixedWing:RES_R1632_ROM
- R34: renamed from R64; footprint RES_R1632_ROM -> FixedWing:RES_R1632_ROM
- R38: renamed from R119; footprint RES_R1632_ROM -> FixedWing:RES_R1632_ROM
- R39: renamed from R65; footprint RES_R1632_ROM -> FixedWing:RES_R1632_ROM
- R4: renamed from R58; footprint RES_R1632_ROM -> FixedWing:RES_R1632_ROM
- R43: renamed from R120; footprint RES_R1632_ROM -> FixedWing:RES_R1632_ROM
- R44: renamed from R66; footprint RES_R1632_ROM -> FixedWing:RES_R1632_ROM
- R48: renamed from R121; footprint RES_R1632_ROM -> FixedWing:RES_R1632_ROM
- R49: renamed from R67; footprint RES_R1632_ROM -> FixedWing:RES_R1632_ROM
- R53: renamed from R122; footprint RES_R1632_ROM -> FixedWing:RES_R1632_ROM
- R54: renamed from R68; footprint RES_R1632_ROM -> FixedWing:RES_R1632_ROM
- R58: renamed from R123; footprint RES_R1632_ROM -> FixedWing:RES_R1632_ROM
- R59: renamed from R69; footprint RES_R1632_ROM -> FixedWing:RES_R1632_ROM
- R8: renamed from R114; footprint RES_R1632_ROM -> FixedWing:RES_R1632_ROM
- R9: renamed from R59; footprint RES_R1632_ROM -> FixedWing:RES_R1632_ROM
- renumbered C79 to C1, C75 to C10, C76 to C11, C77 to C12, C78 to C13, C67 to C2, C68 to C3, C69 to C4, C70 to C5, C71 to C6, C72 to C7, C73 to C8, C74 to C9, J18 to J1, LED16 to LED1, LED25 to LED10, LED26 to LED11, LED27 to LED12, LED17 to LED2, LED18 to LED3, LED19 to LED4, LED20 to LED5, LED21 to LED6, LED22 to LED7, LED23 to LED8, LED24 to LED9, Q15 to Q1, Q24 to Q10, Q25 to Q11, Q26 to Q12, Q16 to Q2, Q17 to Q3, Q18 to Q4, Q19 to Q5, Q20 to Q6, Q21 to Q7, Q22 to Q8, Q23 to Q9, R160 to R1, R129 to R10, R47 to R11, R37 to R12, R130 to R15, R48 to R16, R38 to R17, R27 to R2, R131 to R20, R49 to R21, R39 to R22, R132 to R25, R50 to R26, R40 to R27, R133 to R30, R51 to R31, R41 to R32, R134 to R35, R52 to R36, R42 to R37, R135 to R40, R53 to R41, R43 to R42, R136 to R45, R54 to R46, R44 to R47, R128 to R5, R137 to R50, R55 to R51, R45 to R52, R138 to R55, R46 to R57, R26 to R6, R139 to R60, R57 to R61, R28 to R7, Z12 to Z1, Z9 to Z10, Z10 to Z11, Z11 to Z12, Z1 to Z2, Z2 to Z8, Z8 to Z9
Connections:
- net STACK_TOP: no longer names the net of J1.13, R58.2, R59.2, R60.2, R61.1

Commit message: feat: schematic pretty much done
Connections:
- net C0: no longer Q1.1 (B), R2.2, Z1.1 (K)
- new net: Q1.1 (B), R2.2, Z1.1 (K)
Changed lines of the file:
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@@
   (title_block
     (title "Cell Filtering and Balancing")
-    (date "2024-08-10")
+    (date "2025-01-19")
     (rev "A")
     (company "AeroNU - FixedWing")
@@
   (junction (at 347.98 143.51) (diameter 0) (color 0 0 0 0)
   )
-  (junction (at 30.48 152.4) (diameter 0) (color 0 0 0 0)
-  )
   (junction (at 195.58 143.51) (diameter 0) (color 0 0 0 0)
   )
@@
   (junction (at 360.68 143.51) (diameter 0) (color 0 0 0 0)
   )
-  (junction (at 30.48 160.02) (diameter 0) (color 0 0 0 0)
-  )
   (junction (at 294.64 199.39) (diameter 0) (color 0 0 0 0)
   )
@@
     (stroke (width 0) (type default))
   )
-  (wire (pts (xy 30.48 152.4) (xy 30.48 160.02))
-    (stroke (width 0) (type default))
-  )
   (wire (pts (xy 379.73 85.09) (xy 381 85.09))
     (stroke (width 0) (type default))
@@
   )
   (text_box "NOTE:\nDesign based on section 2.4 (External Cell-Balancing Circuit Design Using BJTs) of the Cell Balancing With BQ769x2 Battery Monitors guide by TI, available at http://www.ti.com/lit/pdf/sluaa81"
-    (at 13.97 257.81 0) (size 160.02 7.62)
+    (at 111.76 255.27 0) (size 194.31 6.35)
     (stroke (width 0) (type default))
     (fill (type none))
-    (effects (font (size 1.27 1.27)) (justify left top))
+    (effects (font (size 1.27 1.27)) (justify left top) (href "http://www.ti.com/lit/pdf/sluaa81"))
   )
   (hierarchical_label "C10" (shape output) (at 347.98 236.22 270) (fields_autoplaced)
@@
   )
   (symbol (lib_id "FixedWing:S13B-XH-A") (at 200.66 35.56 90) (unit 1)
-    (in_bom yes) (on_board yes) (dnp no) (fields_autoplaced)
-    (property "Reference" "J1" (at 215.9 15.24 90)
-      (effects (font (size 1.27 1.27)))
-    )
-    (property "Value" "S13B-XH-A" (at 215.9 17.78 90)
+    (in_bom yes) (on_board yes) (dnp no)
+    (property "Reference" "J1" (at 215.9 16.51 90)
+      (effects (font (size 1.27 1.27)))
+    )
+    (property "Value" "S13B-XH-A" (at 215.9 19.05 90)
       (effects (font (size 1.27 1.27)))
     )
@@
   (symbol (lib_id "power:GND") (at 50.8 215.9 0) (unit 1)
     (in_bom yes) (on_board yes) (dnp no) (fields_autoplaced)
-    (property "Reference" "#PWR05" (at 50.8 222.25 0)
+    (property "Reference" "#PWR02" (at 50.8 222.25 0)
       (effects (font (size 1.27 1.27)) hide)
     )
@@
       (project "bms-board"
         (path "/8a7831d1-a913-4f04-8780-225d2234b41d/95f820cc-7b9f-45ce-aa8e-ca8cb50aec5e"
-          (reference "#PWR05") (unit 1)
+          (reference "#PWR02") (unit 1)
         )
       )
@@
   (symbol (lib_id "power:GND") (at 17.78 215.9 0) (unit 1)
     (in_bom yes) (on_board yes) (dnp no) (fields_autoplaced)
-    (property "Reference" "#PWR04" (at 17.78 222.25 0)
+    (property "Reference" "#PWR01" (at 17.78 222.25 0)
       (effects (font (size 1.27 1.27)) hide)
     )
@@
       (project "bms-board"
         (path "/8a7831d1-a913-4f04-8780-225d2234b41d/95f820cc-7b9f-45ce-aa8e-ca8cb50aec5e"
-          (reference "#PWR04") (unit 1)
-        )
-      )
+          (reference "#PWR01") (unit 1)
+        )
+      )

Commit message: feat: schematic cleanup, continued layout
Connections:
- net C0: now also C2.2
- net C1: now also C2.1; no longer C2.2
- net GND: now also J1.1, Q1.2 (E), R1.1, Z1.2 (A); no longer C2.1
Other:
- moved on the sheet: C1, C10, C11, C12, C13, C2, C3, C4, C5, C6, C7, C8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
