File: bms-kicad-project/SensingConnections.kicad_sch (KiCad schematic)
At the start: 42 parts, among them J10 XT60PW-F, J11 XT60PW-F, J12 1053131303, J13 SM06B-GHS-TB, J14 XT60PW-F, J15 1053131302, J16 1053131302, J17 1053131302, J18 1053131302, J6 XT60PW-F, J7 XT60PW-M, J8 XT60PW-F, J9 5024940670, U7 MCP4726A0T-E/CH, U8 MCP9700AT-E/TT, U9 MCP9700AT-E/TT

Commit message: feat: schematic cleanup, continued layout
Parts:
- removed R120: 5.6k, FixedWing:RESC2012X60N, symbol FixedWing:RK73H2ATTD5601F
- removed R121, R122: 100, RESC2012X50N, symbol FixedWing:CRCW0805100RFKEA
- removed R123: 100k, FixedWing:RESC2012X60N, symbol FixedWing:RC0805FR-07100KL
- removed TP21: TestPoint, TestPoint:TestPoint_Pad_D1.5mm, symbol Connector:TestPoint
- added R120: 8.16k, FixedWing:RC0805N_YAG, symbol FixedWing:RT0805BRD078K16L
- added R121: 475, RESC2012X50N, symbol FixedWing:CRCW0805475RFKEA
- added TP19: TestPoint, TestPoint:TestPoint_Pad_D1.5mm, symbol Connector:TestPoint
- renumbered C70 to C65, C65 to C66, C66 to C69, C69 to C70, J14 to J13, J15 to J14, J13 to J15, R124 to R122, R126 to R123, R125 to R124, R127 to R125, U9 to U8, U8 to U9
Connections:
- net +BATT: now also R120.1, TP19.1
- net GND: now also R121.1; no longer J10.3 (MH1), J10.4 (MH2), J11.3 (MH1), J11.4 (MH2), J6.3 (MH1), J6.4 (MH2), J8.3 (MH1), J8.4 (MH2)
- net at J15.4: now also R120.2, R121.2
- net DACCLK renamed DAC_CLK
- net DACDAT renamed DAC_DAT
- net GNDCUR renamed GNDPWR
- net PIXCLK renamed PIX_CLK
- net PIXDAT renamed PIX_DAT
- no-connect marks 4 -> 12
Other:
- note added: "Battery In"
- note removed: "Battery In and Current Sense"
- moved on the sheet: C65, C67, C68, C69, C70, C71, C72, J15, J7, R122, R123, R124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

Commit message: feat: placing cell filtering/balancing components
Parts:
- H1, H2, H3, H4, H5, H6, H7, H8: footprint MountingHole:MountingHole_3.2mm_M3_Pad_Via -> MountingHole:MountingHole_3.2mm_M3_ISO14580_Pad

Commit message: feat: lotta layout
Parts:
- renumbered J11 to J10, J12 to J11, J13 to J12, J14 to J13, J15 to J14, J16 to J15, J17 to J16, J18 to J17, J6 to J5, J7 to J6, J8 to J7, J9 to J8, J10 to J9, LED15 to LED16, R120 to R121, R121 to R122, R122 to R123, R123 to R124, R124 to R125, R125 to R126

Commit message: feat: big pre-design review schematic commit
Parts:
- added BB1, BB2: Busbar, symbol FixedWing:BUSBAR
- added R127, R128: 10k, FixedWing:KOA_Speer-RK73H2A-0-0-MFG, symbol FixedWing:RK73H2ATTD1002F
- renumbered C66 to C72, C65 to C73, C67 to C74, C68 to C75, C69 to C76, C70 to C77, C71 to C78, C72 to C79, J15 to J14, J16 to J15, J17 to J16, J14 to J17, R121 to R125, R122 to R126, R123 to R129, R124 to R130, R125 to R131, R126 to R132
Connections:
- net +BATT: now also BB1.1
- net DAC_CLK: now also R128.1
- net DAC_DAT: now also R127.1
- net GNDPWR: now also BB2.1
- net +3.3V renamed +3V3
- net +3V3: now also R127.2, R128.2
Other:
- note added: "Busbars"
- company: (none) -> AeroNU - FixedWing
- moved on the sheet: C73, C74, C75, C76, C77, C78, C79, H1, H2, H3, H4, H5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

Commit message: feat: post-design review clarity
Parts:
- added CR2, CR3: USBLC6-2SC6, FixedWing:SOT23-6L_STM, symbol FixedWing:USBLC6-2SC6
- added TP40: ~, TestPoint:TestPoint_Pad_D1.0mm, symbol FixedWing:TestPoint
- BB1: footprint (none) -> FixedWing:BUSBAR_LONG
- BB2: footprint (none) -> FixedWing:BUSBAR_SHORT
- TP39: renamed from TP19; value TestPoint -> ~; footprint TestPoint:TestPoint_Pad_D1.5mm -> TestPoint:TestPoint_Pad_D1.0mm; symbol Connector:TestPoint -> FixedWing:TestPoint
- renumbered J11 to J10, J12 to J11, J8 to J12, J9 to J8, J10 to J9, R127 to R126, R128 to R127, R125 to R128, R126 to R129, R129 to R130, R130 to R131, R131 to R132, R132 to R133
Connections:
- net +5V: now also CR2.5, CR3.5
- net GND: now also CR2.2, CR3.2
- net PIX_CLK: now also CR2.6; no longer J12.3
- net PIX_DAT: now also CR2.4; no longer J12.4
- net RGB_DOUT: now also TP40.1
- net at R128.2, R129.2: now also CR3.4; no longer J17.4
- net at C76.2, U7.1 (VOUT): now also CR3.6; no longer J17.3
- new net: CR2.1, J12.3
- new net: CR2.3, J12.4
- new net: CR3.1, J17.3
- new net: CR3.3, J17.4
Other:
- moved on the sheet: C73, C74, C75, C76, C77, J12, R126, R127, R128, R129, U7

Commit message: feat: I am so tired. 4-layer layout almost done
Parts:
- removed H5, H6, H7, H8: MountingHole_Pad, MountingHole:MountingHole_3.2mm_M3_ISO14580_Pad, symbol Mechanical:MountingHole_Pad
- removed R126, R127: 10k, FixedWing:KOA_Speer-RK73H2A-0-0-MFG, symbol FixedWing:RK73H2ATTD1002F
- added MP1, MP2, MP3, MP4: WA-SMSI_9774XXX360, FixedWing:WA-SMSI_9774150360, symbol FixedWing:WA-SMSI_9774XXX360
- added R126, R127, R128, R129: 5.1k, FixedWing:RESC2012X60N, symbol FixedWing:RC0805JR-075K1L
- renumbered C72 to C81, C73 to C82, C74 to C83, C75 to C84, C76 to C85, C77 to C86, C78 to C87, C79 to C88, R128 to R130, R129 to R131, R130 to R132, R131 to R133, R132 to R134, R133 to R135, TP39 to TP32, TP40 to TP33
Connections:
- net GNDPWR is gone; now on net GND: BB2.1, J11.2, J13.2, J14.2, J15.2, J16.2, J5.2, J7.2, J8.2, J9.2
- net +3V3: now also R126.2, R127.2, R128.2, R129.2
- net DAC_CLK: now also R129.1
- net DAC_DAT: now also R128.1
- net GND: now also MP1.1, MP2.1, MP3.1, MP4.1
- net PIX_CLK: now also R126.1
- net PIX_DAT: now also R127.1
- net TEMP_BAL renamed TEMP_ESC
Other:
- note added: "BMS and ESC Mounting 2x(M3*4)"
- note removed: "ESC and BMS Mounting 2x(M3*4)"
- moved on the sheet: CR2, CR3, H2, H3, H4, J12, R130, R131

Commit message: feat: biiig layout and slight design change commit
Parts:
- removed C88: 1µ, FixedWing:CAPC1608X90N, symbol FixedWing:GCM188R71C105KA64D
- removed MP1, MP2, MP3, MP4: WA-SMSI_9774XXX360, FixedWing:WA-SMSI_9774150360, symbol FixedWing:WA-SMSI_9774XXX360
- removed R133, R135: 100, RESC2012X50N, symbol FixedWing:CRCW0805100RFKEA
- removed U9: MCP9700AT-E/TT, FixedWing:SOT-23_MC_MCH, symbol FixedWing:MCP9700AT-E_TT
- added C84: 0.1µ, FixedWing:CAP_GCJ-18_MUR, symbol FixedWing:GCJ188R72A104KA01D
- added H5, H6, H7: MountingHole_Pad, MountingHole:MountingHole_3.2mm_M3_ISO14580_Pad, symbol Mechanical:MountingHole_Pad
- added Q14: DNBT8105-7, FixedWing:SOT95P240X105-3N, symbol FixedWing:DNBT8105-7
- added R135, R136: 1k, FixedWing:RC0805N_YAG, symbol FixedWing:RC0805FR-071KL
- added X2: PKMCS0909E4000-R1, FixedWing:PKMCS0909E4000-R1_MUR, symbol FixedWing:PKMCS0909E4000-R1
- J11: renamed from J10; Manufacturer (none) -> Molex
- J13: renamed from J12; Manufacturer (none) -> Molex
- J18: renamed from J17; Manufacturer (none) -> JST (JAPAN SOLDERLESS TERMINALS)
- renumbered BB2 to BB1, BB1 to BB2, C84 to C85, C85 to C86, C86 to C87, C87 to C88, J9 to J10, J11 to J12, J13 to J14, J14 to J15, J15 to J16, J16 to J17, J5 to J6, J6 to J7, J7 to J8, J8 to J9, R126 to R127, R127 to R128, R128 to R129, R129 to R130, R130 to R131, R131 to R132, R132 to R133, TP32 to TP31, TP33 to TP32
Connections:
- net TEMP_ESC is gone; now on net TEMP_CORE: U8.2 (VOUT)
- net +5V: now also R136.2, X2.2
- net GND: now also C84.1, H5.1, H6.1, H7.1, Q14.2 (E)
- net at CR3.4, R131.2, R132.2: now also C84.2
- new net: Q14.1 (B), R135.2
- new net: Q14.3 (C), R136.1, X2.1
- new net BUZZ: R135.1
Other:
- note added: "Buzzer"
- note added: "Temperature Sensor"
- note removed: "Temperature Sensors"
- moved on the sheet: BB1, BB2, C88, H1, H2, H3, H4, R131, R132, R133, R134, U8
