File: bms-kicad-project/SensingConnections.kicad_sch (KiCad schematic)
At the start: 3 parts, among them U8 ACS72981KLRATR-150B5

Commit message: Wired up most external connections
Parts:
- added C66: 0.1µ, FixedWing:G-21_MUR, symbol FixedWing:GCM21BR72A104KA37L
- added H1, H2, H3, H4, H5, H6, H7, H8: MountingHole_Pad, MountingHole:MountingHole_3.2mm_M3_Pad_Via, symbol Mechanical:MountingHole_Pad
- added J10, J7, J8, J9: 1053131302, FixedWing:105313YY02, symbol FixedWing:1053131302
- added J11, J12, J13, J14: XT60PW-F, FixedWing:XT60PWF, symbol FixedWing:XT60PW-F
- added J15: 1053131303, FixedWing:105313YY03, symbol FixedWing:1053131303
- added J16: 5024940670, FixedWing:5024940670, symbol FixedWing:5024940670
- added J17: SM06B-GHS-TB, FixedWing:SM06B-GHS-TB, symbol FixedWing:SM06B-GHS-TB_LF__SN_
- added J6: XT60PW-M, FixedWing:XT60PWM, symbol FixedWing:XT60PW-M
- added LED15: COM-16347, FixedWing:COM-16347_SPK, symbol FixedWing:COM-16347
- added R108: 100k, FixedWing:RESC2012X60N, symbol FixedWing:RC0805FR-07100KL
- added R109: 5.6k, FixedWing:RESC2012X60N, symbol FixedWing:RK73H2ATTD5601F
- added R110, R111: 100, RESC2012X50N, symbol FixedWing:CRCW0805100RFKEA
Connections:
- net +5V: now also C66.2, J10.1, J15.1, J16.1, J16.2, J17.1, J17.2, J7.1, J8.1, J9.1, LED15.1 (VDD)
- net +BATT: now also J11.1, J12.1, J13.1, J14.1, R108.2
- net CUR_SENSE: now also J17.3
- net GND: now also C66.1, H1.1, H2.1, H3.1, H4.1, H5.1, H6.1, H7.1, H8.1, J10.2, J11.2, J11.3 (MH1), J11.4 (MH2), J12.2, J12.3 (MH1), J12.4 (MH2), J13.2, J13.3 (MH1), J13.4 (MH2), J14.2, J14.3 (MH1), J14.4 (MH2), J15.3, J16.5, J16.6, J16.MP1, J16.MP2, J17.5, J17.6, J6.1, J6.3, J6.4, J7.2, J8.2, J9.2, LED15.3 (VSS), R109.1
- net at U8.5 (IP+): now also J6.2
- new net: R109.2, R110.1
- new net: R110.2, R111.1
- new net: J15.2, LED15.2 (DOUT)
- new net: J17.4, R108.1, R111.2
- new net LEDOUT: LED15.4 (DIN)
- new net PIXCLK: J16.3
- new net PIXDAT: J16.4
Other:
- note added: "+5V Out"
- note added: "Battery In and Current Sense"
- note added: "Battery Out"
- note added: "ESC and BMS Mounting 2x(M3*4)"
- note added: "Pixhawk Analog Power"
- note added: "Pixhawk Digital Power"
- note added: "RGB LED Out"
- moved on the sheet: C64, C65, U8

Commit message: feat: Just shifting a few things around
Parts:
- renumbered C66 to C64, C64 to C66, J12 to J10, J9 to J11, J13 to J12, J10 to J13, J15 to J14, J14 to J15, J17 to J16, J16 to J17, J11 to J6, J6 to J8, J8 to J9, R109 to R108, R110 to R109, R111 to R110, R108 to R111
Other:
- moved on the sheet: C64, J10, J11, J12, J13, J14, J15, J16, J17, J6, J7, J9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

Commit message: Feature/library migration (#19)
* feat: first library migration commit

* feat: added sims directory, new cell balancing components

* feat: cell filtering/balancing switchover done

* feat: don't even know what I changed, just zoned out for several hours. Made PCB r/a mount XT-60s and solder pads into a 2-for-1 deal

* feat: schematic pretty much done

* feat: started layout

* feat: added current sense DAC

* feat: added capacitors to DAC

* feat:added more capacitors to DAC

* feat: more DAC capacitors

* feat: added temp sensor symbol/footprint

* added temp sense cad models

* feat: Added temp sensors

* feat: schematic cleanup, continued layout

* feat: added tvs protection ic to usb

* feat: placing cell filtering/balancing components

* feat: lotta layout

* feat: cell balancing board

* feat: changed cell balancing schem

* feat: slightly edited cell balance schem

* feat: big pre-design review schematic commit

* feat: post-design review clarity

* feat: I am so tired. 4-layer layout almost done

* feat: biiig layout and slight design change commit

* feat:bos->lax layout sesh

* feat: lax -> syd layout sesh

* feat: DRC run

* feat: deleted manufacturing files

* feat: silkscreen done

* feat: REV A COMMIT FOR FAB

* doc: updated schematic docs

---------

Co-authored-by: Ronan Gleason <gleason.r@northeastern.edu>
Co-authored-by: cassidysakamoto <sakamoto.ca@northeastern.edu>
Parts:
- removed C64, C66: 0.1µ, FixedWing:G-21_MUR, symbol FixedWing:GCM21BR72A104KA37L
- removed C65: 1.5n, FixedWing:G-21_MUR, symbol FixedWing:GRM2165C1H152JA01D
- removed H8: MountingHole_Pad, MountingHole:MountingHole_3.2mm_M3_Pad_Via, symbol Mechanical:MountingHole_Pad
- removed R108: 5.6k, FixedWing:RESC2012X60N, symbol FixedWing:RK73H2ATTD5601F
- removed R109, R110: 100, RESC2012X50N, symbol FixedWing:CRCW0805100RFKEA
- removed R111: 100k, FixedWing:RESC2012X60N, symbol FixedWing:RC0805FR-07100KL
- removed U8: ACS72981KLRATR-150B5, FixedWing:ACS780LLRTR050BT, symbol FixedWing:ACS72981KLRATR-150B5
- added BB1: Busbar, FixedWing:BUSBAR_SHORT, symbol FixedWing:BUSBAR
- added BB2: Busbar, FixedWing:BUSBAR_LONG, symbol FixedWing:BUSBAR
- added C80, C82, C83, C84, C85: 0.1µ, FixedWing:CAP_GCJ-18_MUR, symbol FixedWing:GCJ188R72A104KA01D
- added C81, C86: 10µ, FixedWing:CAP_CL21B106KOQNNNE_SAM, symbol FixedWing:CL21B106KOQNNNE
- added C87: 1µ, FixedWing:CAPC1608X90N, symbol FixedWing:GCM188R71C105KA64D
- added CR2, CR3: USBLC6-2SC6, FixedWing:SOT23-6L_STM, symbol FixedWing:USBLC6-2SC6
- added J10: XT60PW-F, FixedWing:XT60PWF, symbol FixedWing:XT60PW-F
- added Q14: DNBT8105-7, FixedWing:SOT95P240X105-3N, symbol FixedWing:DNBT8105-7
- added R129, R130, R131, R132: 5.1k, FixedWing:RESC2012X60N, symbol FixedWing:RC0805JR-075K1L
- added R133: 8.16k, FixedWing:RC0805N_YAG, symbol FixedWing:RT0805BRD078K16L
- added R134: 475, RESC2012X50N, symbol FixedWing:CRCW0805475RFKEA
- added R135, R136: 100, RESC2012X50N, symbol FixedWing:CRCW0805100RFKEA
- added R137, R138: 1k, FixedWing:RC0805N_YAG, symbol FixedWing:RC0805FR-071KL
- added TP25: ~, TestPoint:TestPoint_Pad_D1.0mm, symbol FixedWing:TestPoint
- added U8: MCP4726A0T-E/CH, FixedWing:SOT-23-6_MC_MCH, symbol FixedWing:MCP4726A0T-E_CH
- added U9: MCP9700AT-E/TT, FixedWing:SOT-23_MC_MCH, symbol FixedWing:MCP9700AT-E_TT
- added X2: PKMCS0909E4000-R1, FixedWing:PKMCS0909E4000-R1_MUR, symbol FixedWing:PKMCS0909E4000-R1
- H1, H2, H3, H4, H5, H6, H7: footprint MountingHole:MountingHole_3.2mm_M3_Pad_Via -> MountingHole:MountingHole_3.2mm_M3_ISO14580_Pad
- J11: renamed from J14; Manufacturer (none) -> Molex
- J12: renamed from J15; footprint FixedWing:XT60PWF -> FixedWing:XT60PWF_Pad; Manufacturer (none) -> Amass
- J13: renamed from J17; Manufacturer (none) -> Molex
- J18: renamed from J16; Manufacturer (none) -> JST (JAPAN SOLDERLESS TERMINALS)
- J6: Manufacturer (none) -> Amass
- J7: renamed from J8; footprint FixedWing:XT60PWM -> FixedWing:XT60PWM_Pad; Manufacturer (none) -> Changzou Amass Elec
- J8: renamed from J10; Manufacturer (none) -> Amass
- J9: renamed from J12; Manufacturer (none) -> Amass
- renumbered J7 to J14, J9 to J15, J11 to J16, J13 to J17, LED15 to LED16
Connections:
- net +5V: now also C80.2, C84.2, C86.2, CR2.5, CR3.5, R135.1, R138.2, U8.3 (VDD), X2.2
- net +BATT: now also J7.2, BB2.1, J10.1, R133.1, TP25.1
- net GND: now also J18.7, J18.8, BB1.1, C80.1, C81.1, C82.1, C83.1, C84.1, C85.1, C86.1, C87.1, CR2.2, CR3.2, J10.2, Q14.2 (E), R134.1, U8.2 (VSS), U9.3 (GND); no longer J12.3 (MH1), J12.4 (MH2), J6.3 (MH1), J6.4 (MH2), J7.1, J7.3, J7.4, J8.3 (MH1), J8.4 (MH2), J9.3 (MH1), J9.4 (MH2)
- net RGB_DOUT: now reaches J11.2, LED16.2 (DOUT)
- net at J18.4: now also CR3.3
- net CUR_SENSE: no longer names the net of J18.3
- net CUR_SENSE: now also CR3.1
- net LEDOUT renamed RGB_DIN
- net PIXCLK: no longer names the net of J13.3
- net PIXCLK: now also CR2.1
- net PIXDAT: no longer names the net of J13.4
- net PIXDAT: now also CR2.3
- new net: C83.2, CR3.4, R133.2, R134.2
- new net: Q14.1 (B), R137.2
- new net: Q14.3 (C), R138.1, X2.1
- new net: R135.2, R136.1
- new net: C85.2, CR3.6, U8.1 (VOUT)
- new net: C87.2, R136.2, U9.1 (VDD)
- new net +3V3: C81.2, C82.2, R129.2, R130.2, R131.2, R132.2, U8.6 (VREF)
- new net -BATT: J7.1
- new net BUZZ: R137.1
- new net DAC_CLK: R132.1, U8.5 (SCL)
- new net DAC_DAT: R131.1, U8.4 (SDA)
- new net PIX_CLK: CR2.6, R129.1
- new net PIX_DAT: CR2.4, R130.1
- new net TEMP_AMB: U9.2 (VOUT)
- no-connect marks 0 -> 12
Other:
- note added: "BMS and ESC Mounting 2x(M3*4)"
- note added: "Battery In"
- note added: "Busbars"
- note added: "Buzzer"
- note added: "DAC"
- note added: "Temperature Sensor"
- note removed: "Battery In and Current Sense"
- note removed: "ESC and BMS Mounting 2x(M3*4)"
- company: (none) -> AeroNU - FixedWing
- title: (none) -> External Connections and Sensing
- moved on the sheet: J11, J12, J13, J14, J15, J16, J17, J6, J7, J8, J9, LED16

Commit message: feat: initial pass at rev. B
Parts:
- removed C80: 0.1µ, FixedWing:CAP_GCJ-18_MUR, symbol FixedWing:GCJ188R72A104KA01D
- removed CR2, CR3: USBLC6-2SC6, FixedWing:SOT23-6L_STM, symbol FixedWing:USBLC6-2SC6
- added C80: 10µ, FixedWing:CAP_CL21B106KOQNNNE_SAM, symbol FixedWing:CL21B106KOQNNNE
- added C95, C96: 0.1µ, FixedWing:CAP_GCJ-18_MUR, symbol FixedWing:GCJ188R72A104KA01D
- added D10, D11, D12, D13, D14, D15, D16, D7: GG0603052R542P, FixedWing:DIONC1608X70N, symbol FixedWing:GG0603052R542P
- added D5, D6, D8, D9: GG060303100N2P, FixedWing:DIONC1608X70N, symbol FixedWing:GG060303100N2P
- added U10: 74LVC1T45W6-7, FixedWing:SOT26-6_DIO, symbol FixedWing:74LVC1T45W6-7
Connections:
- net +3V3: now also C84.2, C86.2, R135.1, U8.3 (VDD), C95.1, U10.1 (VCC(A)), U10.5 (DIR)
- net +5V: now also C80.2, C96.1, D10.1 (A1), D11.1 (A1), D12.1 (A1), D13.1 (A1), D14.1 (A1), D15.1 (A1), D7.1 (A1), U10.6 (VCC(B)); no longer C84.2, C86.2, R135.1, U8.3 (VDD)
- net GND: now also C80.1, C95.2, C96.2, D10.2 (A2), D11.2 (A2), D12.2 (A2), D13.2 (A2), D14.2 (A2), D15.2 (A2), D16.2 (A2), D5.2 (A2), D6.2 (A2), D7.2 (A2), D8.1 (A1), D9.1 (A1), U10.2 (GND)
- net PIX_CLK: now also J13.3, D9.2 (A2)
- net PIX_DAT: now also J13.4, D8.2 (A2)
- net RGB_DIN: now also U10.3 (A); no longer LED16.4 (DIN)
- net RGB_DOUT: now also D16.1 (A1)
- net at C83.2, R133.2, R134.2: now also J18.4, D6.1 (A1)
- net at J18.3: now also C85.2, U8.1 (VOUT), D5.1 (A1)
- new net: LED16.4 (DIN), U10.4 (B)
Other:
- note added: "- Back-Powering +5V And +BATT Rails From +3V3"
- note added: "- RGB LED Logic Level Mismatch"
- moved on the sheet: BB1, BB2, C83, J11, J14, J15, J16, J17, LED16, R130, R133, R134
