File: bms-kicad-project/_autosave-bms-board.kicad_pcb (KiCad board)
At the start: 6 copper layers, 100 x 100 mm, 345 parts, among them J1 S13B-XH-A, J10 1053131303, J11 XT60PW-F, J12 5024940670, J13 1053131302, J14 1053131302, J15 1053131302, J16 1053131302, J17 SM06B-GHS-TB, J18 Conn_01x03, J2 1053141308, J3 12402012E212A, J4 Conn_02x04_Odd_Even, J5 XT60PW-F, J6 XT60PW-M, J7 XT60PW-F, J8 XT60PW-F, J9 XT60PW-F, Q1 DNBT8105-7, Q10 DNBT8105-7, Q11 DNBT8105-7, Q12 DNBT8105-7, Q13 BSS308PE_H6327, Q2 DNBT8105-7, Q3 DNBT8105-7, Q4 DNBT8105-7, Q5 DNBT8105-7, Q6 DNBT8105-7, Q7 DNBT8105-7, Q8 DNBT8105-7, Q9 DNBT8105-7, SW1 KMR223G LFG, SW2 KMR223G LFG, U1 TMUX7208PWR, U2 BQ7697204PFBR, U3 SIC461ED-T1-GE3, U4 W25Q128JVSIQ TR, U5 NCP1117ST33T3G, U6 RP2040, U7 MCP4726A0T-E/CH, U8 MCP9700AT-E/TT, U9 MCP9700AT-E/TT, X1 ABM8-272-T3

Commit message: feat: biiig layout and slight design change commit
Routing:
- net +3V3: track 118.9 -> 119.7 mm, vias 24 -> 22
Changed lines of the file:
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@@
   (segment (start 335.663772 111.875) (end 335.307054 111.518282) (width 0.2) (layer "F.Cu") (net 3))
   (via (at 330.125919 110.986581) (size 0.6) (drill 0.35) (layers "F.Cu" "B.Cu") (remove_unused_layers) (keep_end_layers) (free) (zone_layer_connections "In3.Cu") (net 3))
-  (via (at 330.5 122.3) (size 0.6) (drill 0.35) (layers "F.Cu" "B.Cu") (remove_unused_layers) (keep_end_layers) (zone_layer_connections "In3.Cu") (net 3))
+  (via (at 330.6 122.2) (size 0.6) (drill 0.35) (layers "F.Cu" "B.Cu") (remove_unused_layers) (keep_end_layers) (zone_layer_connections "In3.Cu") (net 3))
   (via (at 336.449 116.6) (size 0.6) (drill 0.35) (layers "F.Cu" "B.Cu") (remove_unused_layers) (keep_end_layers) (free) (zone_layer_connections "In3.Cu") (net 3))
   (via (at 330.2 114.7) (size 0.6) (drill 0.35) (layers "F.Cu" "B.Cu") (remove_unused_layers) (keep_end_layers) (free) (zone_layer_connections "In3.Cu") (net 3))
@@
   (via (at 333.194669 114.055331) (size 0.6) (drill 0.35) (layers "F.Cu" "B.Cu") (remove_unused_layers) (keep_end_layers) (free) (zone_layer_connections "In3.Cu") (net 3))
   (via (at 332 109.6) (size 0.6) (drill 0.35) (layers "F.Cu" "B.Cu") (remove_unused_layers) (keep_end_layers) (free) (zone_layer_connections "In3.Cu") (net 3))
-  (via (at 331.9 122.3) (size 0.6) (drill 0.35) (layers "F.Cu" "B.Cu") (remove_unused_layers) (keep_end_layers) (zone_layer_connections "In3.Cu") (net 3))
-  (via (at 331.9 123.3) (size 0.6) (drill 0.35) (layers "F.Cu" "B.Cu") (remove_unused_layers) (keep_end_layers) (zone_layer_connections "In3.Cu") (net 3))
+  (via (at 331.8 122.2) (size 0.6) (drill 0.35) (layers "F.Cu" "B.Cu") (remove_unused_layers) (keep_end_layers) (zone_layer_connections "In3.Cu") (net 3))
+  (via (at 331.8 123.4) (size 0.6) (drill 0.35) (layers "F.Cu" "B.Cu") (remove_unused_layers) (keep_end_layers) (zone_layer_connections "In3.Cu") (net 3))
   (via (at 341 111.1) (size 0.6) (drill 0.35) (layers "F.Cu" "B.Cu") (remove_unused_layers) (keep_end_layers) (free) (zone_layer_connections "In3.Cu") (net 3))
   (via (at 348.4 111.05) (size 0.6) (drill 0.35) (layers "F.Cu" "B.Cu") (remove_unused_layers) (keep_end_layers) (free) (zone_layer_connections "In3.Cu") (net 3))
-  (via (at 330.5 123.3) (size 0.6) (drill 0.35) (layers "F.Cu" "B.Cu") (remove_unused_layers) (keep_end_layers) (zone_layer_connections "In3.Cu") (net 3))
+  (via (at 330.6 123.4) (size 0.6) (drill 0.35) (layers "F.Cu" "B.Cu") (remove_unused_layers) (keep_end_layers) (zone_layer_connections "In3.Cu") (net 3))
   (via (at 333.2 115.1) (size 0.6) (drill 0.35) (layers "F.Cu" "B.Cu") (remove_unused_layers) (keep_end_layers) (free) (zone_layer_connections "In3.Cu") (net 3))
-  (via (at 331.2 122.8) (size 0.6) (drill 0.35) (layers "F.Cu" "B.Cu") (remove_unused_layers) (keep_end_layers) (zone_layer_connections "In3.Cu") (net 3))
   (via (at 335.307054 111.518282) (size 0.6) (drill 0.35) (layers "F.Cu" "B.Cu") (remove_unused_layers) (keep_end_layers) (free) (zone_layer_connections "In3.Cu") (net 3))
   (via (at 333.2 112.019669) (size 0.6) (drill 0.35) (layers "F.Cu" "B.Cu") (remove_unused_layers) (keep_end_layers) (free) (zone_layer_connections "In3.Cu") (net 3))
@@
   (via (at 373.549 67.524998) (size 0.6) (drill 0.35) (layers "F.Cu" "B.Cu") (free) (net 3))
   (via (at 354.4 125.125) (size 0.6) (drill 0.35) (layers "F.Cu" "B.Cu") (remove_unused_layers) (keep_end_layers) (free) (zone_layer_connections) (net 3))
-  (via (at 327.1 117.6) (size 0.6) (drill 0.35) (layers "F.Cu" "B.Cu") (remove_unused_layers) (keep_end_layers) (zone_layer_connections) (net 3))
   (via (at 345.6 119.925) (size 0.6) (drill 0.35) (layers "F.Cu" "B.Cu") (remove_unused_layers) (keep_end_layers) (free) (zone_layer_connections "In3.Cu") (net 3))
   (segment (start 351.8 108.9) (end 358.3 108.9) (width 1) (layer "In3.Cu") (net 3))
@@
   (segment (start 358.3 108.9) (end 370.3 96.9) (width 1) (layer "In3.Cu") (net 3))
   (segment (start 373.6456 76.187242) (end 373.6456 65.4) (width 1) (layer "In3.Cu") (net 3))
-  (segment (start 321.04 117.65) (end 321 117.61) (width 0.6) (layer "B.Cu") (net 3))
   (segment (start 335.8375 107.526471) (end 334.9 108.463971) (width 0.2) (layer "B.Cu") (net 3))
   (segment (start 335.50364 116.8375) (end 335.3 117.04114) (width 0.2) (layer "B.Cu") (net 3))
+  (segment (start 328.5 117.6) (end 324.94 117.6) (width 0.6) (layer "B.Cu") (net 3))
   (segment (start 341 111.1) (end 341.125 110.975) (width 0.2) (layer "B.Cu") (net 3))
   (segment (start 344.349 118.3) (end 344.2625 118.3) (width 0.2) (layer "B.Cu") (net 3))
@@
   (segment (start 330.1375 110.975) (end 330.4375 110.675) (width 0.2) (layer "B.Cu") (net 3))
   (segment (start 334.9 108.463971) (end 334.9 110.7) (width 0.2) (layer "B.Cu") (net 3))
-  (segment (start 324.89 117.65) (end 321.04 117.65) (width 0.6) (layer "B.Cu") (net 3))
   (segment (start 336 133.935) (end 336 131.4) (width 1) (layer "B.Cu") (net 3))
   (segment (start 344.349 118.298) (end 344.349 118.3) (width 0.2) (layer "B.Cu") (net 3))
   (segment (start 333.2 112.019669) (end 332.9 111.719669) (width 0.2) (layer "B.Cu") (net 3))
+  (segment (start 323.94 118.6) (end 321.99 118.6) (width 0.6) (layer "B.Cu") (net 3))
   (segment (start 331.2 126.6) (end 331.2 122.8) (width 1) (layer "B.Cu") (net 3))
   (segment (start 336 131.4) (end 331.2 126.6) (width 1) (layer "B.Cu") (net 3))
@@
   (segment (start 330.2 114.7) (end 330.6375 115.1375) (width 0.2) (layer "B.Cu") (net 3))
   (segment (start 335.8375 106.25) (end 335.8375 107.526471) (width 0.2) (layer "B.Cu") (net 3))
+  (segment (start 324.94 117.6) (end 323.94 118.6) (width 0.6) (layer "B.Cu") (net 3))
   (segment (start 336.2115 116.8375) (end 335.50364 116.8375) (width 0.2) (layer "B.Cu") (net 3))
   (segment (start 341.125 110.975) (end 342.1375 110.975) (width 0.2) (layer "B.Cu") (net 3))
@@
   (segment (start 335.3 111.511228) (end 335.3 110.7) (width 0.2) (layer "B.Cu") (net 3))
   (segment (start 330.9 108.8) (end 331.2 108.8) (width 0.2) (layer "B.Cu") (net 3))
+  (segment (start 321.99 118.6) (end 321 117.61) (width 0.6) (layer "B.Cu") (net 3))
   (segment (start 335.3 117.04114) (end 335.3 117.575) (width 0.2) (layer "B.Cu") (net 3))
   (segment (start 333.3 110.7) (end 333.3 110.4) (width 0.2) (layer "B.Cu") (net 3))
-  (segment (start 328.5 117.6) (end 324.94 117.6) (width 0.6) (layer "B.Cu") (net 3))
   (segment (start 341.1 115.1375) (end 338.9375 115.1375) (width 0.2) (layer "B.Cu") (net 3))
   (segment (start 338.9 102.6) (end 338.97 102.67) (width 0.2) (layer "B.Cu") (net 3))
@@
   (segment (start 340.5625 111.5375) (end 338.9375 111.5375) (width 0.2) (layer "B.Cu") (net 3))
   (segment (start 333.2 115.1) (end 333.1625 115.1375) (width 0.2) (layer "B.Cu") (net 3))
-  (segment (start 324.94 117.6) (end 324.89 117.65) (width 0.6) (layer "B.Cu") (net 3))
   (segment (start 335.307054 111.518282) (end 335.3 111.511228) (width 0.2) (layer "B.Cu") (net 3))
   (segment (start 346.95 111.05) (end 346.8 111.2) (width 0.2) (layer "B.Cu") (net 3))
