File: bms-kicad-project/5VPower.kicad_sch (KiCad schematic)
At the start: 59 parts, among them Q15 BSS308PE_H6327, Q16 BSS308PE_H6327, U11 LM66100DCKR, U12 LM66100DCKR, U3 SIC461ED-T1-GE3

Commit message: feat: Rev. B release
Parts:
- added D2: GG0603052R542P, FixedWing:DIONC1608X70N, symbol FixedWing:GG0603052R542P
- C90, C91: footprint FixedWing:CAPC2012X140N -> FixedWing:CAPC1608X90N; symbol FixedWing:GCM21BR71C105KA58L -> FixedWing:GCM188R71C105KA64D; Manufacturer Part Number GCM21BR71C105KA58L -> GCM188R71C105KA64D
Connections:
- net 5V_PRE: now also D2.1 (A1)
- net GND: now also D2.2 (A2)
Other:
- moved on the sheet: C90, C91, Q15, Q16, R139, R140, U11, U12
